File: pcb/Duo_Adapter_V0.5/Duo_Adapter_V0.5.kicad_pcb (KiCad board)
At the start: 2 copper layers, 109.2 x 78.7 mm, 67 parts

Commit message: Duo Adapter V0.5
noch nicht fertig
Parts:
- added LP28: Lötpad, Duo:Lötpad_1x02_Buchse, F.Cu at (125.5, 121.9)
- added LP29: Lötpad, Duo:Lötpad_1x02_Buchse, F.Cu at (128.0, 121.9)
- added LP30: Lötpad, Duo:Lötpad_1x02_Buchse, F.Cu at (130.6, 121.9)
- added LP31: Lötpad, Duo:Lötpad_1x02_Buchse, F.Cu at (133.1, 121.9)
- added U1: 74HC4050, Duo:DIP-16__300, F.Cu at (131.1, 99.6)
Routing:
- net GND: track 154.5 -> 192.9 mm
- net +3V3: track 2.54 -> 40.6 mm
- net Net-(LP28-Pad2): track 0.00 -> 34.5 mm
- net Net-(LP29-Pad2): track 0.00 -> 28.9 mm
- net Net-(LP28-Pad1): track 0.00 -> 28.6 mm
- net Net-(LP30-Pad2): track 0.00 -> 24.9 mm
- net Net-(LP29-Pad1): track 0.00 -> 23.5 mm
- net Net-(LP30-Pad1): track 0.00 -> 19.7 mm
- net Net-(LP31-Pad2): track 0.00 -> 19.5 mm
- net Net-(LP31-Pad1): track 0.00 -> 12.9 mm
