File: pcb/megashield_svn_1.3_geoeffnet/Bohrlöcher.sch (KiCad schematic (older format))
At the start: 18 parts

Commit message: Platine V1.3
Hierarchischer Schaltplan für Step Down Wandler erstellt
Parts:
- B1, B15, B16, B17, B18, B2, B3, B4, B5, B6, B7, B8: footprint (none) -> ACS712:Bohrloch_3,2mm
- B10, B11, B12, B13, B14, B9: footprint (none) -> ACS712:Bohrloch_6,5mm
Changed lines of the file:
@@
 EESchema Schematic File Version 2
+LIBS:Lötpad_2,5mm
 LIBS:power
 LIBS:Bluetooth_ZS_HC_05
@@
 $Descr A4 11693 8268
 encoding utf-8
-Sheet 14 16
+Sheet 14 17
 Title "Ardumower shield SVN Version 1.3"
 Date "Sonntag, 26. April 2015"
 Rev "1.3"
-Comp " by UweZ"
+Comp "von UweZ"
 Comment1 ""
 Comment2 ""
@@
 F 0 "B1" H 1225 1225 60  0000 C CNN
 F 1 "Bohrloch_3,2mm" H 1175 1145 60  0000 C CNN
-F 2 "" H 945 1065 60  0000 C CNN
+F 2 "ACS712:Bohrloch_3,2mm" H 945 1065 60  0001 C CNN
 F 3 "" H 945 1065 60  0000 C CNN
 	1    945  1065
@@
 F 0 "B2" H 1225 1500 60  0000 C CNN
 F 1 "Bohrloch_3,2mm" H 1175 1420 60  0000 C CNN
-F 2 "" H 945 1340 60  0000 C CNN
+F 2 "ACS712:Bohrloch_3,2mm" H 945 1340 60  0001 C CNN
 F 3 "" H 945 1340 60  0000 C CNN
 	1    945  1340
@@
 F 0 "B3" H 1225 1765 60  0000 C CNN
 F 1 "Bohrloch_3,2mm" H 1175 1685 60  0000 C CNN
-F 2 "" H 945 1605 60  0000 C CNN
+F 2 "ACS712:Bohrloch_3,2mm" H 945 1605 60  0001 C CNN
 F 3 "" H 945 1605 60  0000 C CNN
 	1    945  1605
@@
 F 0 "B4" H 1225 2035 60  0000 C CNN
 F 1 "Bohrloch_3,2mm" H 1175 1955 60  0000 C CNN
-F 2 "" H 945 1875 60  0000 C CNN
+F 2 "ACS712:Bohrloch_3,2mm" H 945 1875 60  0001 C CNN
 F 3 "" H 945 1875 60  0000 C CNN
 	1    945  1875
@@
 F 0 "B5" H 2100 1225 60  0000 C CNN
 F 1 "Bohrloch_3,2mm" H 2050 1145 60  0000 C CNN
-F 2 "" H 1820 1065 60  0000 C CNN
+F 2 "ACS712:Bohrloch_3,2mm" H 1820 1065 60  0001 C CNN
 F 3 "" H 1820 1065 60  0000 C CNN
 	1    1820 1065
@@
 F 0 "B6" H 2100 1500 60  0000 C CNN
 F 1 "Bohrloch_3,2mm" H 2050 1420 60  0000 C CNN
-F 2 "" H 1820 1340 60  0000 C CNN
+F 2 "ACS712:Bohrloch_3,2mm" H 1820 1340 60  0001 C CNN
 F 3 "" H 1820 1340 60  0000 C CNN
 	1    1820 1340
@@
 F 0 "B7" H 2100 1765 60  0000 C CNN
 F 1 "Bohrloch_3,2mm" H 2050 1685 60  0000 C CNN
-F 2 "" H 1820 1605 60  0000 C CNN
+F 2 "ACS712:Bohrloch_3,2mm" H 1820 1605 60  0001 C CNN
 F 3 "" H 1820 1605 60  0000 C CNN
 	1    1820 1605
@@
 F 0 "B8" H 2100 2035 60  0000 C CNN
 F 1 "Bohrloch_3,2mm" H 2050 1955 60  0000 C CNN
-F 2 "" H 1820 1875 60  0000 C CNN
+F 2 "ACS712:Bohrloch_3,2mm" H 1820 1875 60  0001 C CNN
 F 3 "" H 1820 1875 60  0000 C CNN
 	1    1820 1875
@@
 F 0 "B15" H 3035 1230 60  0000 C CNN
 F 1 "Bohrloch_3,2mm" H 2985 1150 60  0000 C CNN
-F 2 "" H 2755 1070 60  0000 C CNN
+F 2 "ACS712:Bohrloch_3,2mm" H 2755 1070 60  0001 C CNN
 F 3 "" H 2755 1070 60  0000 C CNN
 	1    2755 1070
@@
 F 0 "B16" H 3035 1505 60  0000 C CNN
 F 1 "Bohrloch_3,2mm" H 2985 1425 60  0000 C CNN
-F 2 "" H 2755 1345 60  0000 C CNN
+F 2 "ACS712:Bohrloch_3,2mm" H 2755 1345 60  0001 C CNN
 F 3 "" H 2755 1345 60  0000 C CNN
 	1    2755 1345
@@
 F 0 "B17" H 3035 1770 60  0000 C CNN
 F 1 "Bohrloch_3,2mm" H 2985 1690 60  0000 C CNN
-F 2 "" H 2755 1610 60  0000 C CNN
+F 2 "ACS712:Bohrloch_3,2mm" H 2755 1610 60  0001 C CNN
 F 3 "" H 2755 1610 60  0000 C CNN
 	1    2755 1610
@@
 F 0 "B18" H 3035 2040 60  0000 C CNN
 F 1 "Bohrloch_3,2mm" H 2985 1960 60  0000 C CNN
-F 2 "" H 2755 1880 60  0000 C CNN
+F 2 "ACS712:Bohrloch_3,2mm" H 2755 1880 60  0001 C CNN
 F 3 "" H 2755 1880 60  0000 C CNN
 	1    2755 1880
@@
 F 0 "B12" H 4195 1230 60  0000 C CNN
 F 1 "Bohrloch_6,5mm" H 4145 1150 60  0000 C CNN
-F 2 "" H 3915 1070 60  0000 C CNN
+F 2 "ACS712:Bohrloch_6,5mm" H 3915 1070 60  0001 C CNN
 F 3 "" H 3915 1070 60  0000 C CNN
 	1    3915 1070
@@
 F 0 "B13" H 4195 1505 60  0000 C CNN
 F 1 "Bohrloch_6,5mm" H 4145 1425 60  0000 C CNN
-F 2 "" H 3915 1345 60  0000 C CNN
+F 2 "ACS712:Bohrloch_6,5mm" H 3915 1345 60  0001 C CNN
 F 3 "" H 3915 1345 60  0000 C CNN
 	1    3915 1345
@@
 F 0 "B14" H 4195 1770 60  0000 C CNN
 F 1 "Bohrloch_6,5mm" H 4145 1690 60  0000 C CNN
-F 2 "" H 3915 1610 60  0000 C CNN
+F 2 "ACS712:Bohrloch_6,5mm" H 3915 1610 60  0001 C CNN
 F 3 "" H 3915 1610 60  0000 C CNN
 	1    3915 1610
@@
 $EndComp
 $Comp
-L GND #PWR0134
+L GND #PWR0121
 U 1 1 553D45B9
 P 3820 1070
-F 0 "#PWR0134" H 3820 820 60  0001 C CNN
+F 0 "#PWR0121" H 3820 820 60  0001 C CNN
 F 1 "GND" V 3820 855 60  0000 C CNN
 F 2 "" H 3820 1070 60  0000 C CNN
@@
 $EndComp
 $Comp
-L GND #PWR0135
+L GND #PWR0122
 U 1 1 553D46A2
 P 3820 1345
-F 0 "#PWR0135" H 3820 1095 60  0001 C CNN
+F 0 "#PWR0122" H 3820 1095 60  0001 C CNN
 F 1 "GND" V 3820 1130 60  0000 C CNN
 F 2 "" H 3820 1345 60  0000 C CNN
@@
 $EndComp
 $Comp
-L GND #PWR0136
+L GND #PWR0123
 U 1 1 553D46E4
 P 3820 1610
-F 0 "#PWR0136" H 3820 1360 60  0001 C CNN
+F 0 "#PWR0123" H 3820 1360 60  0001 C CNN
 F 1 "GND" V 3820 1395 60  0000 C CNN
 F 2 "" H 3820 1610 60  0000 C CNN
@@
 F 0 "B9" H 5305 1225 60  0000 C CNN
 F 1 "Bohrloch_6,5mm" H 5255 1145 60  0000 C CNN
-F 2 "" H 5025 1065 60  0000 C CNN
+F 2 "ACS712:Bohrloch_6,5mm" H 5025 1065 60  0001 C CNN
 F 3 "" H 5025 1065 60  0000 C CNN
 	1    5025 1065
@@
 F 0 "B10" H 5305 1500 60  0000 C CNN
 F 1 "Bohrloch_6,5mm" H 5255 1420 60  0000 C CNN
-F 2 "" H 5025 1340 60  0000 C CNN
+F 2 "ACS712:Bohrloch_6,5mm" H 5025 1340 60  0001 C CNN
 F 3 "" H 5025 1340 60  0000 C CNN
 	1    5025 1340
@@
 F 0 "B11" H 5305 1765 60  0000 C CNN
 F 1 "Bohrloch_6,5mm" H 5255 1685 60  0000 C CNN
-F 2 "" H 5025 1605 60  0000 C CNN
+F 2 "ACS712:Bohrloch_6,5mm" H 5025 1605 60  0001 C CNN
 F 3 "" H 5025 1605 60  0000 C CNN
 	1    5025 1605
