File: pcb/megashield_svn_1.3_geoeffnet/Dropsensor.sch (KiCad schematic (older format))
At the start: 4 parts, among them P21 DropRight, P31 DropLeft

Commit message: Platine V1.3
Hierarchischer Schaltplan für Step Down Wandler erstellt
Parts:
- D5, D6: footprint (none) -> ACS712:Diode_ligend_RM10
- P21, P31: footprint (none) -> ACS712:Pin_Header_Straight_1x03
Changed lines of the file:
@@
 EESchema Schematic File Version 2
+LIBS:Lötpad_2,5mm
 LIBS:power
 LIBS:Bluetooth_ZS_HC_05
@@
 $Descr A4 11693 8268
 encoding utf-8
-Sheet 9 16
+Sheet 9 17
 Title "Ardumower shield SVN Version 1.3"
 Date "Sonntag, 26. April 2015"
 Rev "1.3"
-Comp " by UweZ"
-Comment1 ""
+Comp "von UweZ"
+Comment1 "Dropsensoren"
 Comment2 ""
 Comment3 ""
@@
 F 0 "P31" V 4215 2425 50  0000 C CNN
 F 1 "DropLeft" V 4315 2425 40  0000 C CNN
-F 2 "" H 4265 2425 60  0000 C CNN
+F 2 "ACS712:Pin_Header_Straight_1x03" H 4265 2425 60  0001 C CNN
 F 3 "" H 4265 2425 60  0000 C CNN
 F 4 "Value" H 4265 2425 60  0001 C CNN "Bestellnummer"
@@
 $EndComp
 $Comp
-L GND #PWR068
+L GND #PWR055
 U 1 1 553C96A2
 P 4820 2425
-F 0 "#PWR068" H 4820 2175 60  0001 C CNN
+F 0 "#PWR055" H 4820 2175 60  0001 C CNN
 F 1 "GND" V 4820 2205 60  0000 C CNN
 F 2 "" H 4820 2425 60  0000 C CNN
@@
 $EndComp
 $Comp
-L +5V #PWR069
+L +5V #PWR056
 U 1 1 553C96B7
 P 4820 2325
-F 0 "#PWR069" H 4820 2175 60  0001 C CNN
+F 0 "#PWR056" H 4820 2175 60  0001 C CNN
 F 1 "+5V" V 4820 2540 60  0000 C CNN
 F 2 "" H 4820 2325 60  0000 C CNN
@@
 F 0 "D5" H 5330 2625 40  0000 C CNN
 F 1 "1N4148" H 5330 2425 40  0000 C CNN
-F 2 "" H 5330 2525 60  0000 C CNN
+F 2 "ACS712:Diode_ligend_RM10" H 5330 2525 60  0001 C CNN
 F 3 "" H 5330 2525 60  0000 C CNN
 	1    5330 2525
@@
 F 0 "P21" V 4210 2925 50  0000 C CNN
 F 1 "DropRight" V 4310 2925 40  0000 C CNN
-F 2 "" H 4260 2925 60  0000 C CNN
+F 2 "ACS712:Pin_Header_Straight_1x03" H 4260 2925 60  0001 C CNN
 F 3 "" H 4260 2925 60  0000 C CNN
 F 4 "Value" H 4260 2925 60  0001 C CNN "Bestellnummer"
@@
 $EndComp
 $Comp
-L GND #PWR070
+L GND #PWR057
 U 1 1 553CC968
 P 4815 2925
-F 0 "#PWR070" H 4815 2675 60  0001 C CNN
+F 0 "#PWR057" H 4815 2675 60  0001 C CNN
 F 1 "GND" V 4815 2705 60  0000 C CNN
 F 2 "" H 4815 2925 60  0000 C CNN
@@
 $EndComp
 $Comp
-L +5V #PWR071
+L +5V #PWR058
 U 1 1 553CC96E
 P 4815 2825
-F 0 "#PWR071" H 4815 2675 60  0001 C CNN
+F 0 "#PWR058" H 4815 2675 60  0001 C CNN
 F 1 "+5V" V 4815 3040 60  0000 C CNN
 F 2 "" H 4815 2825 60  0000 C CNN
@@
 F 0 "D6" H 5325 3125 40  0000 C CNN
 F 1 "1N4148" H 5325 2925 40  0000 C CNN
-F 2 "" H 5325 3025 60  0000 C CNN
+F 2 "ACS712:Diode_ligend_RM10" H 5325 3025 60  0001 C CNN
 F 3 "" H 5325 3025 60  0000 C CNN
 	1    5325 3025
