File: pcb/megashield_svn_1.3_geoeffnet/INA169.sch (KiCad schematic (older format))
At the start: 6 parts, among them U4 INA169_IC

Commit message: Platine V1.3
Einzelne Bauteile auf SMD angepasst
Belegung Anschlussstecker geändert +5V und GND
Anschlussstecker auf KK Stecker umgeändert
Parts:
- C14: Bauform (none) -> 1206; Bestelllink (none) -> https://www.reichelt.de/X7R-G1206-100N/3/index.html?&ACTION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; Bestellnummer (none) -> R: X7R-G1206 100N; Technische Daten (none) -> Vielschicht-Keramikkondensator 100N, 10% 63V
- JP12: renamed from JP?; footprint (none) -> ACS712:Pin_Header_Straight_1x02
- U4: footprint ina169_breakout:ina169_ic_sot23-5 -> Housings_SOT-23_SOT-143_TSOT-6:SOT-23-5
Changed lines of the file:
@@
 $Descr A4 11693 8268
 encoding utf-8
-Sheet 26 27
+Sheet 26 25
 Title ""
 Date ""
@@
 F 2 "Capacitors_SMD:C_1206" H 7308 3150 30  0001 C CNN
 F 3 "" H 7270 3300 60  0000 C CNN
+F 4 "Vielschicht-Keramikkondensator 100N, 10% 63V" H 7270 3300 60  0001 C CNN "Technische Daten"
+F 5 "R: X7R-G1206 100N" H 7270 3300 60  0001 C CNN "Bestellnummer"
+F 6 "1206" H 7270 3300 60  0001 C CNN "Bauform"
+F 7 "https://www.reichelt.de/X7R-G1206-100N/3/index.html?&ACTION=3&LA=446&ARTICLE=22889&artnr=X7R-G1206+100N&SEARCH=X7R-G1206" H 7270 3300 60  0001 C CNN "Bestelllink"
 	1    7270 3300
 	1    0    0    -1
@@
 F 0 "U4" H 6460 2650 60  0000 C CNN
 F 1 "INA169_IC" H 6460 2050 60  0000 C CNN
-F 2 "ina169_breakout:ina169_ic_sot23-5" H 6460 2050 60  0001 C CNN
+F 2 "Housings_SOT-23_SOT-143_TSOT-6:SOT-23-5" H 6460 2050 60  0001 C CNN
 F 3 "" H 6460 2050 60  0000 C CNN
 F 4 "Value" H 6460 2350 60  0001 C CNN "Technische Daten"
@@
 	5020 2300 5020 3900
 $Comp
-L JUMPER JP?
+L JUMPER JP12
 U 1 1 55EE25EF
 P 5665 3550
-F 0 "JP?" H 5665 3700 60  0000 C CNN
+F 0 "JP12" H 5665 3700 60  0000 C CNN
 F 1 "Messbereich 5A/2,5A" H 5665 3470 40  0000 C CNN
-F 2 "" H 5665 3550 60  0000 C CNN
+F 2 "ACS712:Pin_Header_Straight_1x02" H 5665 3550 60  0001 C CNN
 F 3 "" H 5665 3550 60  0000 C CNN
 	1    5665 3550
