File: pcb/Test_und_Entwicklung/megashield_svn_1.3_geoeffnet/Wlan_BT_Uhr_IMU.sch (KiCad schematic (older format))
At the start: 12 parts, among them P44 Wlan, P5 GPS, U11 Wlan_ESP8266, U2 Bluetooth_CZ_HC_05

Commit message: megashield_svn_1.3_geoeffnet
Zwischenschritt Sicherheitscopie
Parts:
- P44, P5: footprint Pin_Headers:Pin_Header_Straight_1x05 -> Zimprich:JST_EH_B05B-EH-A_05x2.50mm_Straight
Changed lines of the file:
@@
 LIBS:conn
 LIBS:transistors
+LIBS:cmos_ieee
+LIBS:cmos4000
+LIBS:switches
 LIBS:ardumower mega shield svn-cache
 EELAYER 25 0
@@
 $Descr A3 16535 11693
 encoding utf-8
-Sheet 8 24
+Sheet 8 25
 Title "Ardumower shield SVN Version"
-Date "29 Dez 2014"
-Rev "1.2"
-Comp "SM & UZ"
+Date "2016-09-30"
+Rev "1.3"
+Comp "ML AG JL UZ"
 Comment1 ""
 Comment2 ""
@@
 NoConn ~ 6475 2535
 $Comp
-L GND #PWR44
+L GND #PWR040
 U 1 1 57DCCA39
 P 6695 2335
-F 0 "#PWR44" H 6695 2085 50  0001 C CNN
+F 0 "#PWR040" H 6695 2085 50  0001 C CNN
 F 1 "GND" V 6695 2135 50  0000 C CNN
 F 2 "" H 6695 2335 50  0000 C CNN
@@
 $EndComp
 $Comp
-L GND #PWR54
+L GND #PWR041
 U 1 1 57DCD18B
 P 7900 5470
-F 0 "#PWR54" H 7900 5220 50  0001 C CNN
+F 0 "#PWR041" H 7900 5220 50  0001 C CNN
 F 1 "GND" H 7905 5297 50  0000 C CNN
 F 2 "" H 7900 5470 50  0000 C CNN
@@
 $EndComp
 $Comp
-L GND #PWR52
+L GND #PWR042
 U 1 1 57DCD73B
 P 7800 2185
-F 0 "#PWR52" H 7800 1935 50  0001 C CNN
+F 0 "#PWR042" H 7800 1935 50  0001 C CNN
 F 1 "GND" V 7800 1985 50  0000 C CNN
 F 2 "" H 7800 2185 50  0000 C CNN
@@
 $EndComp
 $Comp
-L GND #PWR43
+L GND #PWR043
 U 1 1 57DE0935
 P 6680 4995
-F 0 "#PWR43" H 6680 4745 50  0001 C CNN
+F 0 "#PWR043" H 6680 4745 50  0001 C CNN
 F 1 "GND" V 6680 4795 50  0000 C CNN
 F 2 "" H 6680 4995 50  0000 C CNN
@@
 F 0 "P44" H 8137 2326 50  0000 L CNN
 F 1 "Wlan" H 8137 2235 50  0000 L CNN
-F 2 "Pin_Headers:Pin_Header_Straight_1x05" H 8138 2348 50  0001 L CNN
+F 2 "Zimprich:JST_EH_B05B-EH-A_05x2.50mm_Straight" H 8138 2348 50  0001 L CNN
 F 3 "" H 8060 2285 50  0001 C CNN
 F 4 "Value" H 8138 2249 60  0001 L CNN "Gehäuseart"
@@
 $EndBitmap
 $Comp
-L +3.3VP #PWR50
+L +3.3VP #PWR044
 U 1 1 57E9FA66
 P 7785 2485
-F 0 "#PWR50" H 7935 2435 50  0001 C CNN
+F 0 "#PWR044" H 7935 2435 50  0001 C CNN
 F 1 "+3.3VP" V 7780 2585 50  0000 L CNN
 F 2 "" H 7785 2485 50  0000 C CNN
@@
 $EndComp
 $Comp
-L +5VP #PWR51
+L +5VP #PWR045
 U 1 1 57E9FA6C
 P 7800 2085
-F 0 "#PWR51" H 7800 1935 50  0001 C CNN
+F 0 "#PWR045" H 7800 1935 50  0001 C CNN
 F 1 "+5VP" V 7800 2295 50  0000 C CNN
 F 2 "" H 7800 2085 50  0000 C CNN
@@
 $EndComp
 $Comp
-L +3.3VP #PWR42
+L +3.3VP #PWR046
 U 1 1 57EA0D72
 P 6535 2235
-F 0 "#PWR42" H 6685 2185 50  0001 C CNN
+F 0 "#PWR046" H 6685 2185 50  0001 C CNN
 F 1 "+3.3VP" V 6530 2335 50  0000 L CNN
 F 2 "" H 6535 2235 50  0000 C CNN
@@
 $EndComp
 $Comp
-L +3.3VP #PWR41
+L +3.3VP #PWR047
 U 1 1 57EA0FE0
 P 6535 2035
-F 0 "#PWR41" H 6685 1985 50  0001 C CNN
+F 0 "#PWR047" H 6685 1985 50  0001 C CNN
 F 1 "+3.3VP" V 6530 2135 50  0000 L CNN
 F 2 "" H 6535 2035 50  0000 C CNN
@@
 $EndComp
 $Comp
-L +5VP #PWR45
+L +5VP #PWR048
 U 1 1 57EA1F8B
 P 6765 5470
-F 0 "#PWR45" H 6765 5320 50  0001 C CNN
+F 0 "#PWR048" H 6765 5320 50  0001 C CNN
 F 1 "+5VP" V 6765 5680 50  0000 C CNN
 F 2 "" H 6765 5470 50  0000 C CNN
@@
 $EndComp
 $Comp
-L +3.3VP #PWR47
+L +3.3VP #PWR049
 U 1 1 57EA255C
 P 7265 5445
-F 0 "#PWR47" H 7415 5395 50  0001 C CNN
+F 0 "#PWR049" H 7415 5395 50  0001 C CNN
 F 1 "+3.3VP" V 7260 5545 50  0000 L CNN
 F 2 "" H 7265 5445 50  0000 C CNN
@@
 $EndComp
 $Comp
-L +3.3VP #PWR48
+L +3.3VP #PWR050
 U 1 1 57EA2CC1
 P 7280 4695
-F 0 "#PWR48" H 7430 4645 50  0001 C CNN
+F 0 "#PWR050" H 7430 4645 50  0001 C CNN
 F 1 "+3.3VP" V 7275 4795 50  0000 L CNN
 F 2 "" H 7280 4695 50  0000 C CNN
@@
 $EndComp
 $Comp
-L GND #PWR46
+L GND #PWR051
 U 1 1 57EA782C
 P 7185 3215
-F 0 "#PWR46" H 7185 2965 50  0001 C CNN
+F 0 "#PWR051" H 7185 2965 50  0001 C CNN
 F 1 "GND" V 7185 3015 50  0000 C CNN
 F 2 "" H 7185 3215 50  0000 C CNN
@@
 F 0 "P5" H 11348 3636 50  0000 L CNN
 F 1 "GPS" H 11348 3545 50  0000 L CNN
-F 2 "Pin_Headers:Pin_Header_Straight_1x05" H 11270 3595 50  0001 C CNN
+F 2 "Zimprich:JST_EH_B05B-EH-A_05x2.50mm_Straight" H 11270 3595 50  0001 C CNN
 F 3 "" H 11270 3595 50  0000 C CNN
 F 4 "Value" H 11270 3595 60  0001 C CNN "Gehäuseart"
@@
 $EndComp
 $Comp
-L +3.3VP #PWR55
+L +3.3VP #PWR052
 U 1 1 57EB99EB
 P 11530 3795
-F 0 "#PWR55" H 11680 3745 50  0001 C CNN
+F 0 "#PWR052" H 11680 3745 50  0001 C CNN
 F 1 "+3.3VP" V 11525 3895 50  0000 L CNN
 F 2 "" H 11530 3795 50  0000 C CNN
@@
 	11530 3795 11470 3795
 $Comp
-L GND #PWR57
+L GND #PWR053
 U 1 1 57EBA23F
 P 11670 3495
-F 0 "#PWR57" H 11670 3245 50  0001 C CNN
+F 0 "#PWR053" H 11670 3245 50  0001 C CNN
 F 1 "GND" V 11670 3295 50  0000 C CNN
 F 2 "" H 11670 3495 50  0000 C CNN
@@
 $EndComp
 $Comp
-L +5VP #PWR53
+L +5VP #PWR054
 U 1 1 57EBB2DC
 P 7830 1935
-F 0 "#PWR53" H 7830 1785 50  0001 C CNN
+F 0 "#PWR054" H 7830 1785 50  0001 C CNN
 F 1 "+5VP" V 7830 2145 50  0000 C CNN
 F 2 "" H 7830 1935 50  0000 C CNN
@@
 $EndComp
 $Comp
-L +5VP #PWR49
+L +5VP #PWR055
 U 1 1 57EBB965
 P 7475 5485
-F 0 "#PWR49" H 7475 5335 50  0001 C CNN
+F 0 "#PWR055" H 7475 5335 50  0001 C CNN
 F 1 "+5VP" H 7475 5650 50  0000 C CNN
 F 2 "" H 7475 5485 50  0000 C CNN
@@
 $EndComp
 $Comp
-L +5VP #PWR56
+L +5VP #PWR056
 U 1 1 57EBF820
 P 11670 3395
-F 0 "#PWR56" H 11670 3245 50  0001 C CNN
+F 0 "#PWR056" H 11670 3245 50  0001 C CNN
 F 1 "+5VP" V 11670 3605 50  0000 C CNN
 F 2 "" H 11670 3395 50  0000 C CNN

Commit message: megashield_svn_1.3_geoeffnet
megashield_svn_1.3_geoeffnet Sicherheitscopie
Parts:
- R14, R15, R16, R6, R7, R8: footprint Resistors_SMD:R_1206 -> Resistors_SMD:R_0805
Changed lines of the file:
@@
 1B AD C3 34 17 14 41 5C 13 18 40 36 55 49 23 66 36 62 24 B8 6F C0 08 96 81 3C 90 04 23 CB DA 25
 0F D4 D6 CE AC 92 3C E3 26 E0 1F 00 19 86 D0 65 A1 44 8A 88 00 00 00 00 49 45 4E 44 AE 42 60 82
-40
+10
 EndData
 $EndBitmap
@@
 13 AB 66 08 3D 82 F4 ED 6A 33 FC 72 2F EA 75 21 FA 55 EB 37 CF 19 F7 FA 0C CF 26 5C CD 56 65 55
 56 82 BC 1E 8F 96 55 59 95 25 96 55 35 5B 95 55 39 E4 F2 FF 01 E2 E8 02 51 02 3C 3A 9F 00 00 00
-00 49 45 4E 44 AE 42 60 82 00
+00 49 45 4E 44 AE 42 60 82 04
 EndData
 $EndBitmap
@@
 F 0 "R6" H 8398 5191 50  0000 L CNN
 F 1 "470R" H 8398 5100 50  0000 L CNN
-F 2 "Resistors_SMD:R_1206" V 8240 5145 50  0001 C CNN
+F 2 "Resistors_SMD:R_0805" V 8240 5145 50  0001 C CNN
 F 3 "Value" H 8310 5145 50  0001 C CNN
 F 4 "Value" H 8398 5266 60  0001 L CNN "Gehäuseart"
@@
 F 0 "R7" H 7988 5191 50  0000 L CNN
 F 1 "1K" H 7988 5100 50  0000 L CNN
-F 2 "Resistors_SMD:R_1206" V 7830 5145 50  0001 C CNN
+F 2 "Resistors_SMD:R_0805" V 7830 5145 50  0001 C CNN
 F 3 "Value" H 7900 5145 50  0001 C CNN
 F 4 "Value" H 7988 5266 60  0001 L CNN "Gehäuseart"
@@
 F 0 "R8" H 7563 5196 50  0000 L CNN
 F 1 "1K" H 7563 5105 50  0000 L CNN
-F 2 "Resistors_SMD:R_1206" V 7405 5150 50  0001 C CNN
+F 2 "Resistors_SMD:R_0805" V 7405 5150 50  0001 C CNN
 F 3 "Value" H 7475 5150 50  0001 C CNN
 F 4 "Value" H 7563 5271 60  0001 L CNN "Gehäuseart"
@@
 F 0 "R15" H 6883 3001 50  0000 L CNN
 F 1 "470R" H 6883 2910 50  0000 L CNN
-F 2 "Resistors_SMD:R_1206" V 6725 2955 50  0001 C CNN
+F 2 "Resistors_SMD:R_0805" V 6725 2955 50  0001 C CNN
 F 3 "Value" H 6795 2955 50  0001 C CNN
 F 4 "Value" H 6883 3076 60  0001 L CNN "Gehäuseart"
@@
 F 0 "R16" H 7273 3011 50  0000 L CNN
 F 1 "1K" H 7273 2920 50  0000 L CNN
-F 2 "Resistors_SMD:R_1206" V 7115 2965 50  0001 C CNN
+F 2 "Resistors_SMD:R_0805" V 7115 2965 50  0001 C CNN
 F 3 "Value" H 7185 2965 50  0001 C CNN
 F 4 "Value" H 7273 3086 60  0001 L CNN "Gehäuseart"
@@
 F 0 "R14" V 7615 1895 50  0000 L CNN
 F 1 "1K" V 7553 1890 50  0000 L CNN
-F 2 "Resistors_SMD:R_1206" V 7395 1935 50  0001 C CNN
+F 2 "Resistors_SMD:R_0805" V 7395 1935 50  0001 C CNN
 F 3 "Value" H 7465 1935 50  0001 C CNN
 F 4 "Value" H 7553 2056 60  0001 L CNN "Gehäuseart"

Commit message: megashield_svn_1.3_geoeffnet
megashield_svn_1.3_geoeffnet sik Kopie
Parts:
- removed R14, R16, R7, R8: 1K, Resistors_SMD:R_0805, symbol R
- removed R15, R6: 470R, Resistors_SMD:R_0805, symbol R
- added JP?: Blue5V/3.3V, Pin_Headers:Pin_Header_Straight_1x03, symbol JUMPER3
- added JP?: Key, Pin_Headers:Pin_Header_Straight_1x02, symbol Jumper_NC_Small
- added Q? (x4): BSS138, TO_SOT_Packages_SMD:SOT-23, symbol BSS138
- added R? (x8): 10K, Resistors_SMD:R_0805, symbol R
Connections:
- net +3.3VP: now also JP?.3; no longer U11.CH_P (CH_PD), U11.VCC
- net +5VP: now also JP?.1
- net GND: now also JP?.2
- net RX1: now also Q?.2 (S), R?.2; no longer P44.3 (P3), U11.TX
- net RX2: now also Q?.2 (S), R?.2; no longer U2.TXD
- net TX1: now also Q?.2 (S), R?.2
- net TX2: now also Q?.2 (S), R?.2
- net at P44.4 (P4), U11.RX: now also Q?.3 (D), R?.2
- net at U11.GP_0 (GP_IO0): now also JP?.1
- net at U2.RXD: now also Q?.3 (D), R?.2
- net at JP4.2, U2.VCC: now also R?.1, R?.1
- new net: P44.3 (P3), Q?.3 (D), R?.2, U11.TX
- new net: JP?.2, R?.1, R?.1, U11.CH_P (CH_PD), U11.VCC
- new net: Q?.3 (D), R?.2, U2.TXD
- new net IOREF: Q?.1 (G), Q?.1 (G), Q?.1 (G), Q?.1 (G), R?.1, R?.1, R?.1, R?.1
- no-connect marks 2 -> 1
Other:
- note added: "Konntrolieren ob Footprint und Lib passt"
- note removed: "Spannungszuordnung prüfen\neinmal vom Arduino und den \nDc Wandlern die Spannungen\nob richtig verdrahtet\n"
- moved on the sheet: JP2, JP4, P44, P5, U11, U2
