File: pcb/Test_und_Entwicklung/megashield_svn_1.3_geoeffnet/Motortreiber.sch (KiCad schematic (older format))
At the start: 9 parts, among them P36 Res24V-2, P39 Res24V-1

Commit message: megashield_svn_1.3_geoeffnet
Alte Version der 1.3 gelöscht und neue Version hochgeladen.
Parts:
- removed C10, C11: 10uF / 63V, Capacitors_SMD:c_elec_6.3x5.8, symbol CP1
- removed CC2, CC3: 100nF 10%, Capacitors_SMD:C_0805, symbol Kondensator
- removed P36: Res24V-2, ACS712:Anschlussklemme_2P_RM5,08, symbol CONN_2
- removed P39: Res24V-1, ACS712:Anschlussklemme_2P_RM5,08, symbol CONN_2
- added P15: Left, Terminal_Blocks:TerminalBlock_Pheonix_MKDS1.5-2pol, symbol CONN_01X02
- added P16, P17: V.OUT, Terminal_Blocks:TerminalBlock_Pheonix_MKDS1.5-2pol, symbol CONN_01X02
- added P18: Right, Terminal_Blocks:TerminalBlock_Pheonix_MKDS1.5-2pol, symbol CONN_01X02
- added P36: Res24V-2, Terminal_Blocks:TerminalBlock_Pheonix_MKDS1.5-2pol, symbol CONN_01X02
- added P37: Mower, Zimprich:Anschlussklemme_RM5,08-RM7,62, symbol CONN_01X02
- added P39: Res24V-1, Terminal_Blocks:TerminalBlock_Pheonix_MKDS1.5-2pol, symbol CONN_01X02
- Dual1, Dual2: footprint ACS712:MC_33926_31polig_mit_Bohrloch_neue_Masse_mit_zweite_Lochreihe -> Zimprich:MC_33926_31polig_mit_Bohrloch_neue_Masse_mit_zweite_Lochreihe; Bestelllink (none) -> Value; Gehäuseart (none) -> Value
- JP16: footprint ACS712:Pin_Header_Straight_1x02 -> Pin_Headers:Pin_Header_Straight_1x02; Bestelllink (none) -> Value; Bestellnummer Value -> (none); Gehäuseart (none) -> Value
Connections:
- net labels added: IOREF
- net labels removed: +5V
- wire segments 64 -> 100
Other:
- note added: "https://www.schukat.com/schukat/schukat_cms_de.nsf/index/CMSDF15D356B046D53BC1256D550038A9E0?OpenDocument&wg=V3672&refDoc=CMS12B13E45BB196811C1257A6A002C97CA\n\nhttps://www.infineon.com/cms/packages/SMD_-_Surface_Mounted_Devices/P-PG-TO252/P-PG-TO252-03-023.html?__locale=de_AT"

Commit message: megashield_svn_1.3_geoeffnet
Zwischenschritt Sicherheitscopie
Parts:
- JP3: renamed from JP16; footprint Pin_Headers:Pin_Header_Straight_1x02 -> Zimprich:Lötpad0,508_CU
Changed lines of the file:
@@
 LIBS:conn
 LIBS:transistors
+LIBS:cmos_ieee
+LIBS:cmos4000
+LIBS:switches
 LIBS:ardumower mega shield svn-cache
 EELAYER 25 0
@@
 $Descr A4 11693 8268
 encoding utf-8
-Sheet 2 24
+Sheet 2 25
 Title "Ardumower shield SVN Version"
-Date "2016-09-25"
-Rev "1.21"
+Date "2016-09-30"
+Rev "1.3"
 Comp "ML AG JL UZ"
 Comment1 ""
@@
 ReserveAD6
 $Comp
-L JUMPER JP16
+L JUMPER JP3
 U 1 1 57D96C22
 P 2795 4975
-F 0 "JP16" H 2790 4815 60  0000 C CNN
+F 0 "JP3" H 2790 4815 60  0000 C CNN
 F 1 "M1FB" H 2795 4895 40  0000 C CNN
-F 2 "Pin_Headers:Pin_Header_Straight_1x02" H 2795 4975 60  0001 C CNN
+F 2 "Zimprich:Lötpad0,508_CU" H 2795 4975 60  0001 C CNN
 F 3 "" H 2795 4975 60  0001 C CNN
 F 4 "Value" H 2795 4975 60  0001 C CNN "Gehäuseart"
@@
 	2495 4975 2425 4975
 $Comp
-L GND #PWR18
+L GND #PWR010
 U 1 1 57DCB31A
 P 7305 2190
-F 0 "#PWR18" H 7305 1940 50  0001 C CNN
+F 0 "#PWR010" H 7305 1940 50  0001 C CNN
 F 1 "GND" V 7305 1995 50  0000 C CNN
 F 2 "" H 7305 2190 50  0000 C CNN
@@
 $EndComp
 $Comp
-L GND #PWR14
+L GND #PWR011
 U 1 1 57DCB496
 P 3510 3025
-F 0 "#PWR14" H 3510 2775 50  0001 C CNN
+F 0 "#PWR011" H 3510 2775 50  0001 C CNN
 F 1 "GND" V 3510 2830 50  0000 C CNN
 F 2 "" H 3510 3025 50  0000 C CNN
@@
 $EndComp
 $Comp
-L GND #PWR13
+L GND #PWR012
 U 1 1 57DCB679
 P 3510 2525
-F 0 "#PWR13" H 3510 2275 50  0001 C CNN
+F 0 "#PWR012" H 3510 2275 50  0001 C CNN
 F 1 "GND" V 3510 2330 50  0000 C CNN
 F 2 "" H 3510 2525 50  0000 C CNN
@@
 $EndComp
 $Comp
-L GND #PWR12
+L GND #PWR013
 U 1 1 57DCB703
 P 3510 1625
-F 0 "#PWR12" H 3510 1375 50  0001 C CNN
+F 0 "#PWR013" H 3510 1375 50  0001 C CNN
 F 1 "GND" V 3510 1430 50  0000 C CNN
 F 2 "" H 3510 1625 50  0000 C CNN
@@
 $EndComp
 $Comp
-L GND #PWR15
+L GND #PWR014
 U 1 1 57DCB93A
 P 3510 4275
-F 0 "#PWR15" H 3510 4025 50  0001 C CNN
+F 0 "#PWR014" H 3510 4025 50  0001 C CNN
 F 1 "GND" V 3510 4080 50  0000 C CNN
 F 2 "" H 3510 4275 50  0000 C CNN
@@
 $EndComp
 $Comp
-L GND #PWR11
+L GND #PWR015
 U 1 1 57DCBAED
 P 3330 5175
-F 0 "#PWR11" H 3330 4925 50  0001 C CNN
+F 0 "#PWR015" H 3330 4925 50  0001 C CNN
 F 1 "GND" V 3330 4980 50  0000 C CNN
 F 2 "" H 3330 5175 50  0000 C CNN
@@
 $EndComp
 $Comp
-L GND #PWR16
+L GND #PWR016
 U 1 1 57DCBBA3
 P 3510 5675
-F 0 "#PWR16" H 3510 5425 50  0001 C CNN
+F 0 "#PWR016" H 3510 5425 50  0001 C CNN
 F 1 "GND" V 3510 5480 50  0000 C CNN
 F 2 "" H 3510 5675 50  0000 C CNN
@@
 $EndComp
 $Comp
-L +24V #PWR17
+L +24V #PWR017
 U 1 1 57DE17A6
 P 7305 2055
-F 0 "#PWR17" H 7305 1905 50  0001 C CNN
+F 0 "#PWR017" H 7305 1905 50  0001 C CNN
 F 1 "+24V" V 7305 2265 50  0000 C CNN
 F 2 "" H 7305 2055 50  0000 C CNN
@@
 $EndSheet
 $Comp
-L +24V #PWR19
+L +24V #PWR018
 U 1 1 57DC0DAD
 P 7735 4665
-F 0 "#PWR19" H 7735 4515 50  0001 C CNN
+F 0 "#PWR018" H 7735 4515 50  0001 C CNN
 F 1 "+24V" V 7735 4875 50  0000 C CNN
 F 2 "" H 7735 4665 50  0000 C CNN
@@
 	7600 4665 7735 4665
 $Comp
-L GND #PWR20
+L GND #PWR019
 U 1 1 57DC2092
 P 7735 4840
-F 0 "#PWR20" H 7735 4590 50  0001 C CNN
+F 0 "#PWR019" H 7735 4590 50  0001 C CNN
 F 1 "GND" V 7735 4645 50  0000 C CNN
 F 2 "" H 7735 4840 50  0000 C CNN
@@
 	5385 4725 5385 4675
 $Comp
-L GND #PWR26
+L GND #PWR020
 U 1 1 57DC50B6
 P 10310 1730
-F 0 "#PWR26" H 10310 1480 50  0001 C CNN
+F 0 "#PWR020" H 10310 1480 50  0001 C CNN
 F 1 "GND" V 10310 1535 50  0000 C CNN
 F 2 "" H 10310 1730 50  0000 C CNN
@@
 $EndComp
 $Comp
-L +24V #PWR25
+L +24V #PWR021
 U 1 1 57DC50BC
 P 10310 1630
-F 0 "#PWR25" H 10310 1480 50  0001 C CNN
+F 0 "#PWR021" H 10310 1480 50  0001 C CNN
 F 1 "+24V" V 10310 1840 50  0000 C CNN
 F 2 "" H 10310 1630 50  0000 C CNN
@@
 	10445 1730 10310 1730
 $Comp
-L GND #PWR28
+L GND #PWR022
 U 1 1 57DC5B70
 P 10315 1095
-F 0 "#PWR28" H 10315 845 50  0001 C CNN
+F 0 "#PWR022" H 10315 845 50  0001 C CNN
 F 1 "GND" V 10315 900 50  0000 C CNN
 F 2 "" H 10315 1095 50  0000 C CNN
@@
 $EndComp
 $Comp
-L +24V #PWR27
+L +24V #PWR023
 U 1 1 57DC5B76
 P 10315 995
-F 0 "#PWR27" H 10315 845 50  0001 C CNN
+F 0 "#PWR023" H 10315 845 50  0001 C CNN
 F 1 "+24V" V 10315 1205 50  0000 C CNN
 F 2 "" H 10315 995 50  0000 C CNN
@@
 	10450 1095 10315 1095
 $Comp
-L GND #PWR22
+L GND #PWR024
 U 1 1 57DC69C8
 P 8850 2225
-F 0 "#PWR22" H 8850 1975 50  0001 C CNN
+F 0 "#PWR024" H 8850 1975 50  0001 C CNN
 F 1 "GND" V 8850 2030 50  0000 C CNN
 F 2 "" H 8850 2225 50  0000 C CNN
@@
 $EndComp
 $Comp
-L +24V #PWR21
+L +24V #PWR025
 U 1 1 57DC69CE
 P 8850 2125
-F 0 "#PWR21" H 8850 1975 50  0001 C CNN
+F 0 "#PWR025" H 8850 1975 50  0001 C CNN
 F 1 "+24V" V 8850 2335 50  0000 C CNN
 F 2 "" H 8850 2125 50  0000 C CNN
@@
 	8985 2225 8850 2225
 $Comp
-L GND #PWR24
+L GND #PWR026
 U 1 1 57DC73F4
 P 8860 4850
-F 0 "#PWR24" H 8860 4600 50  0001 C CNN
+F 0 "#PWR026" H 8860 4600 50  0001 C CNN
 F 1 "GND" V 8860 4655 50  0000 C CNN
 F 2 "" H 8860 4850 50  0000 C CNN
@@
 $EndComp
 $Comp
-L +24V #PWR23
+L +24V #PWR027
 U 1 1 57DC73FA
 P 8860 4750
-F 0 "#PWR23" H 8860 4600 50  0001 C CNN
+F 0 "#PWR027" H 8860 4600 50  0001 C CNN
 F 1 "+24V" V 8860 4960 50  0000 C CNN
 F 2 "" H 8860 4750 50  0000 C CNN

Commit message: megashield_svn_1.3_geoeffnet
megashield_svn_1.3_geoeffnet sik Kopie
Changed lines of the file:
@@
 Sheet 2 25
 Title "Ardumower shield SVN Version"
-Date "2016-09-30"
+Date "2016-10-28"
 Rev "1.3"
 Comp "ML AG JL UZ"
@@
 	0    1    -1   0
 $EndComp
-$Comp
-L +24V #PWR017
-U 1 1 57DE17A6
-P 7305 2055
-F 0 "#PWR017" H 7305 1905 50  0001 C CNN
-F 1 "+24V" V 7305 2265 50  0000 C CNN
-F 2 "" H 7305 2055 50  0000 C CNN
-F 3 "" H 7305 2055 50  0000 C CNN
-	1    7305 2055
-	0    1    -1   0
-$EndComp
 $Sheet
-S 6055 3985 1120 355
+S 6055 3985 1120 455
 U 57DAEC1D
 F0 "MähmotorSchutz" 60
@@
 F4 "MotorOUT1" I R 7175 4280 60
 F5 "MotorOUT2" I R 7175 4080 60
+F6 "+24V" I R 7175 4385 60
 $EndSheet
 Wire Wire Line
@@
 Connection ~ 5565 4275
 $Sheet
-S 5610 2605 1120 355
+S 5610 2605 1120 495
 U 57DB3A39
 F0 "MotorLinks" 60
@@
 F4 "MotorOUT1" I R 6730 2860 60
 F5 "MotorOUT2" I R 6730 2660 60
+F6 "+24V" I R 6730 3010 60
 $EndSheet
 Wire Wire Line
@@
 	6860 2860 6730 2860
 $Sheet
-S 5640 1350 1120 355
+S 5640 1350 1120 460
 U 57DB6176
 F0 "MotorRechts" 60
@@
 F4 "MotorOUT1" I R 6760 1625 60
 F5 "MotorOUT2" I R 6760 1425 60
+F6 "+24V" I R 6760 1745 60
 $EndSheet
 Wire Wire Line
@@
 F5 "Dual1_OUT_GND" I L 6050 4875 60
 $EndSheet
-$Comp
-L +24V #PWR018
-U 1 1 57DC0DAD
-P 7735 4665
-F 0 "#PWR018" H 7735 4515 50  0001 C CNN
-F 1 "+24V" V 7735 4875 50  0000 C CNN
-F 2 "" H 7735 4665 50  0000 C CNN
-F 3 "" H 7735 4665 50  0000 C CNN
-	1    7735 4665
-	0    1    -1   0
-$EndComp
 Wire Wire Line
 	7600 4665 7735 4665
 $Comp
-L GND #PWR019
+L GND #PWR017
 U 1 1 57DC2092
 P 7735 4840
-F 0 "#PWR019" H 7735 4590 50  0001 C CNN
+F 0 "#PWR017" H 7735 4590 50  0001 C CNN
 F 1 "GND" V 7735 4645 50  0000 C CNN
 F 2 "" H 7735 4840 50  0000 C CNN
@@
 	5385 4725 5385 4675
 $Comp
-L GND #PWR020
+L GND #PWR018
 U 1 1 57DC50B6
 P 10310 1730
-F 0 "#PWR020" H 10310 1480 50  0001 C CNN
+F 0 "#PWR018" H 10310 1480 50  0001 C CNN
 F 1 "GND" V 10310 1535 50  0000 C CNN
 F 2 "" H 10310 1730 50  0000 C CNN
@@
 	0    1    -1   0
 $EndComp
-$Comp
-L +24V #PWR021
-U 1 1 57DC50BC
-P 10310 1630
-F 0 "#PWR021" H 10310 1480 50  0001 C CNN
-F 1 "+24V" V 10310 1840 50  0000 C CNN
-F 2 "" H 10310 1630 50  0000 C CNN
-F 3 "" H 10310 1630 50  0000 C CNN
-	1    10310 1630
-	0    -1   -1   0
-$EndComp
 Wire Wire Line
 	10445 1630 10310 1630
@@
 	10445 1730 10310 1730
 $Comp
-L GND #PWR022
+L GND #PWR019
 U 1 1 57DC5B70
 P 10315 1095
-F 0 "#PWR022" H 10315 845 50  0001 C CNN
+F 0 "#PWR019" H 10315 845 50  0001 C CNN
 F 1 "GND" V 10315 900 50  0000 C CNN
 F 2 "" H 10315 1095 50  0000 C CNN
@@
 	0    1    -1   0
 $EndComp
-$Comp
-L +24V #PWR023
-U 1 1 57DC5B76
-P 10315 995
-F 0 "#PWR023" H 10315 845 50  0001 C CNN
-F 1 "+24V" V 10315 1205 50  0000 C CNN
-F 2 "" H 10315 995 50  0000 C CNN
-F 3 "" H 10315 995 50  0000 C CNN
-	1    10315 995
-	0    -1   -1   0
-$EndComp
 Wire Wire Line
 	10450 995  10315 995
@@
 	10450 1095 10315 1095
 $Comp
-L GND #PWR024
+L GND #PWR020
 U 1 1 57DC69C8
 P 8850 2225
-F 0 "#PWR024" H 8850 1975 50  0001 C CNN
+F 0 "#PWR020" H 8850 1975 50  0001 C CNN
 F 1 "GND" V 8850 2030 50  0000 C CNN
 F 2 "" H 8850 2225 50  0000 C CNN
@@
 	0    1    -1   0
 $EndComp
-$Comp
-L +24V #PWR025
-U 1 1 57DC69CE
-P 8850 2125
-F 0 "#PWR025" H 8850 1975 50  0001 C CNN
-F 1 "+24V" V 8850 2335 50  0000 C CNN
-F 2 "" H 8850 2125 50  0000 C CNN
-F 3 "" H 8850 2125 50  0000 C CNN
-	1    8850 2125
-	0    -1   -1   0
-$EndComp
 Wire Wire Line
 	8985 2125 8850 2125
@@
 	8985 2225 8850 2225
 $Comp
-L GND #PWR026
+L GND #PWR021
 U 1 1 57DC73F4
 P 8860 4850
-F 0 "#PWR026" H 8860 4600 50  0001 C CNN
+F 0 "#PWR021" H 8860 4600 50  0001 C CNN
 F 1 "GND" V 8860 4655 50  0000 C CNN
 F 2 "" H 8860 4850 50  0000 C CNN
@@
 	1    8860 4850
 	0    1    -1   0
-$EndComp
-$Comp
-L +24V #PWR027
-U 1 1 57DC73FA
-P 8860 4750
-F 0 "#PWR027" H 8860 4600 50  0001 C CNN
-F 1 "+24V" V 8860 4960 50  0000 C CNN
-F 2 "" H 8860 4750 50  0000 C CNN
-F 3 "" H 8860 4750 50  0000 C CNN
-	1    8860 4750
-	0    -1   -1   0
 $EndComp
 Wire Wire Line
@@
 Text Notes 1100 6255 0    60   ~ 0
 https://www.schukat.com/schukat/schukat_cms_de.nsf/index/CMSDF15D356B046D53BC1256D550038A9E0?OpenDocument&wg=V3672&refDoc=CMS12B13E45BB196811C1257A6A002C97CA\n\nhttps://www.infineon.com/cms/packages/SMD_-_Surface_Mounted_Devices/P-PG-TO252/P-PG-TO252-03-023.html?__locale=de_AT
+Text HLabel 7735 4665 2    50   Input ~ 0
++24V
+Text HLabel 8860 4750 0    50   Input ~ 0
++24V
+Text HLabel 8850 2125 0    50   Input ~ 0
++24V
+Text HLabel 10310 1630 0    50   Input ~ 0
++24V
+Text HLabel 10315 995  0    50   Input ~ 0
++24V
+Text HLabel 7305 2055 2    50   Input ~ 0
++24V
+Text HLabel 6925 1745 2    50   Input ~ 0
++24V
+Wire Wire Line
+	6925 1745 6760 1745
+Text HLabel 6895 3010 2    50   Input ~ 0
++24V
+Wire Wire Line
+	6895 3010 6730 3010
+Wire Wire Line
+	7175 4385 7310 4385
+Text HLabel 7310 4385 2    50   Input ~ 0
++24V
 $EndSCHEMATC

Commit message: megashield_svn_1.3_geoeffnet
Verschiedene 3D Ansichten hinzugefügt
Wlan und BT Modul weiter nach innen verschoben damit es nicht in Kontakt
mit dem Aluprofiel kommt.
Leiterbahnen umgelegt
Footprints und LIb BEzeichnungen Aktualusiert. Kicad hat einige
Footprintordner und Namen umbenann so das die entsprechenden Footprints
nicht mehr gefunden worden
Parts:
- JP3: footprint Zimprich:Lötpad0,508_CU -> Zimprich:SJ; symbol JUMPER -> Jumper
Changed lines of the file:
@@
 LIBS:switches
 LIBS:rfcom
-LIBS:ardumower mega shield svn-cache
 EELAYER 26 0
 EELAYER END
@@
 ReserveAD6
 $Comp
-L JUMPER JP3
+L Jumper JP3
 U 1 1 57D96C22
 P 2795 4975
 F 0 "JP3" H 2790 4815 60  0000 C CNN
 F 1 "M1FB" H 2795 4895 40  0000 C CNN
-F 2 "Zimprich:Lötpad0,508_CU" H 2795 4975 60  0001 C CNN
+F 2 "Zimprich:SJ" H 2795 4975 60  0001 C CNN
 F 3 "" H 2795 4975 60  0001 C CNN
 F 4 "Value" H 2795 4975 60  0001 C CNN "Gehäuseart"
