File: pcb/Test_und_Entwicklung/megashield_svn_1.3_geoeffnet/LShifter2.sch (KiCad schematic (older format))
At the start: 3 parts, among them Q6 BSS138

Commit message: megashield_svn_1.3_geoeffnet
megashield_svn_1.3_geoeffnet
Diverse Änderungen
Schutzschaltung teilweise entfernt
300 Ohm Widerstand eingefügt
9V Pinleite hinzugefügt - wir über das Laderelais geschaltet
Leiterbahnen teileweise neu verlegt
Beidseitiges GND Flächengitter hinzugefügt
Levelschifter Ultraschall Trigger hinzugefügt
usw.....
Parts:
- R60, R61: footprint Resistors_SMD:R_0805 -> Zimprich:R_0603
Changed lines of the file:
@@
 $Descr A4 11693 8268
 encoding utf-8
-Sheet 12 28
+Sheet 12 31
 Title "Ardumower shield SVN Version"
-Date "2016-10-28"
+Date "2017-02-17"
 Rev "1.3"
 Comp "ML AG JL UZ"
@@
 F 0 "R61" H 6198 3296 50  0000 L CNN
 F 1 "10K" H 6198 3205 50  0000 L CNN
-F 2 "Resistors_SMD:R_0805" V 6040 3250 50  0001 C CNN
+F 2 "Zimprich:R_0603" V 6040 3250 50  0001 C CNN
 F 3 "Value" H 6110 3250 50  0001 C CNN
 F 4 "Value" H 6198 3371 60  0001 L CNN "Gehäuseart"
@@
 F 0 "R60" H 5523 3296 50  0000 L CNN
 F 1 "10K" H 5523 3205 50  0000 L CNN
-F 2 "Resistors_SMD:R_0805" V 5365 3250 50  0001 C CNN
+F 2 "Zimprich:R_0603" V 5365 3250 50  0001 C CNN
 F 3 "Value" H 5435 3250 50  0001 C CNN
 F 4 "Value" H 5523 3371 60  0001 L CNN "Gehäuseart"
@@
 $EndComp
 $Comp
-L +5VP #PWR0114
+L +5VP #PWR0115
 U 1 1 57FA81D9
 P 6110 2900
-F 0 "#PWR0114" H 6110 2750 50  0001 C CNN
+F 0 "#PWR0115" H 6110 2750 50  0001 C CNN
 F 1 "+5VP" H 6125 3073 50  0000 C CNN
 F 2 "" H 6110 2900 50  0000 C CNN

Commit message: megashield_svn_1.3_geoeffnet
Alternativer Platz für Summer hinzu gefügt. - Unterhalb des Mega auf der
Rückseite der Platine.
Der Hauptsummer sitzt evl auf der Rückseite hinter dem Bumperduino
ungünstig weil er abgedeckt wird
Parts:
- Q6: symbol BSS138 -> BSS138-RESCUE-ardumower_mega_shield_svn
Changed lines of the file:
@@
 IOREF
 $Comp
-L BSS138 Q6
+L BSS138-RESCUE-ardumower_mega_shield_svn Q6
 U 1 1 57EB0618
 P 5805 3635
@@
 $EndComp
 $Comp
-L +5VP #PWR0130
+L +5VP #PWR0131
 U 1 1 57FA81D9
 P 6110 2900
-F 0 "#PWR0130" H 6110 2750 50  0001 C CNN
+F 0 "#PWR0131" H 6110 2750 50  0001 C CNN
 F 1 "+5VP" H 6125 3073 50  0000 C CNN
 F 2 "" H 6110 2900 50  0000 C CNN
