File: pcb/Test_und_Entwicklung/Sunray_Platinen_Entwicklung_V3 _Serie/ArduSATELino V3.00APD_geoeffnet/ArduSATELino.sch (KiCad schematic (older format))
At the start: 29 parts

Commit message: ArduSATELino V3.00APD_geoeffnet
ArduSATELino V3.00APD_geoeffnet
Parts:
- removed C? (x2): 27pF, Capacitors_SMD:C_0805, symbol C_Small
- removed C? (x2): 10uF, Capacitors_Elko_ThroughHole:Elko_vert_11x5mm_RM2.5, symbol CP_Small
- removed C? (x4): 100nF, Capacitors_SMD:C_0805, symbol C_Small
- removed DIGITAL?: DIGITAL, Pin_Headers:Pin_Header_Straight_1x05, symbol CONN_01X05
- removed IC?: ATMEGA1284-P, DIL40, symbol ATMEGA1284-P
- removed ICSP?: ICSP, Pin_Headers:Pin_Header_Straight_2x03, symbol CONN_02X03
- removed J?: J4, Pin_Headers:Pin_Header_Straight_1x06, symbol CONN_01X06
- removed L?: 10uH, Resistors_ThroughHole:Resistor_Horizontal_RM10mm, symbol L_Small
- removed Q?: 16MHz, Crystals:Crystal_HC49-U_Vertical, symbol Crystal_Small
- removed R?: 1K, Resistors_SMD:R_1206, symbol R_Small
- removed R? (x4): 100, Resistors_SMD:R_1206, symbol R_Small
- removed RS232-TTL?: RS232-TTL, Pin_Headers:Pin_Header_Straight_1x05, symbol CONN_01X05
- removed SJ? (x2): Jumper_NC_Small, Pin_Headers:Pin_Header_Straight_1x02, symbol Jumper_NC_Small
- removed SW?: Reset, Buttons_Switches_SMD:SW_SPST_FSMSM, symbol SW_PUSH
- removed TWI?: TWI, Pin_Headers:Pin_Header_Straight_1x05, symbol CONN_01X05
- added C? (x4): 100nF, symbol C_Small
- added C?: 10uF, symbol C_Small
- added C?: 220uF, symbol CP_Small
- added D? (x6): LED, symbol LED_Small
- added D?: 1N 4004 SMD, Diodes_SMD:DO-214AB, symbol D
- added JP? (x2): Key, Pin_Headers:Pin_Header_Straight_1x02, symbol Jumper_NC_Small
- added JP?: Rst, Pin_Headers:Pin_Header_Straight_1x02, symbol Jumper_NC_Small
- added P?: CONN_01X02, symbol CONN_01X02
- added Q? (x2): BC817-40, SOT-23, symbol BC817-40
- added Q? (x6): BSS138, TO_SOT_Packages_SMD:SOT-23, symbol BSS138
- added R? (x6): 220, Resistors_SMD:R_1206, symbol R_Small
- added R?: 100k, Resistors_SMD:R_1206, symbol R_Small
- added R? (x10): 10k, Resistors_SMD:R_1206, symbol R_Small
- added R? (x4): 10K, Resistors_SMD:R_0805, symbol R
- added SHIELD?: ARDUINO_NANO, symbol ARDUINO_NANO
- added U?: ESP-12E, symbol ESP-12E
- added U?: Wlan_ESP8266, Zimprich:Wlan_ESP8266_3D_mit_Pin_Beschreibung, symbol Wlan_ESP8266_mit_Beschriftung
- added U?: Bluetooth_CZ_HC_05, Zimprich:Bluetooth_Buchse_Platz_mit_Beschriftung, symbol Bluetooth_CZ_HC_05_mit_Beschriftung
- added U?: TSR_1-2433, Converters_DCDC_ACDC:DCDC-Conv_TRACO_TSR-1, symbol TSR_1-2433
- added U?: LM2940CS-3.3, TO254P1435X464-4N, symbol LM2940CS-3.3
Connections:
- net labels added: EXTON, GPIO4, GPIO5, GPIO6, HSPICLK, HSPICSN, HSPIMISO, HSPIMOSI, IRQ, LSPICLK, LSPICSN, LSPIMISO, LSPIMOSI, Led-BT, Led-Wlan, RSTN, RX1, RX2, SYNC, TX1, TX2, WAKEUP
- net labels removed: D3, D4, D5, D6, MISO, MOSI, RXD_TTL, Reset, SCK, SCL, SDA, TXD_TTL, VUSB
- wire segments 82 -> 162
- no-connect marks 1 -> 17
Other:
- note added: "Fällt weg wenn es nicht gebraucht wird"
- note added: "Programmierschaltung for Wlan\nSchaltung im Internet gefunden"
- note added: "[14:15:25] Frederic Goddeeris: It is a ledstrip with WS8212 leds.\nEach led has its own RGB driver.\nBy sending 3 bytes to it, you can control the led, when you send more the next bytes are forwardedn to the next led. This way one can control up to 32 leds with just one output pin. Here I plan to use the different leds to show conenction to AP, c;lient connection, RSSI info?, RX and TX \nhttps://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"
- note added: "https://github.com/FredericG-BE/ardumower/wiki/Using-ESP8266-WIFI-module-on-Ardumower\nBy adding a LED, it is easy to see the state of the ESP8266 firmware: \nconnecting to the WIFI Access Point, Connected, PFOD connected,\n ... Also here, perhaps a LED and resistor could be added directly to the ESP8266 PCB.\nObserve that the GIO bins can only source 12mA.\n I used a 220 Ohm resistor, which will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"
- moved on the sheet: B?, U?
