File: pcb/Produzierte_Platinen/sender_v2_geschlossen/Perimeter sender v2.sch (KiCad schematic (older format))
At the start: 27 parts, among them P1 Vin 24V, P2 VOut 24V, P3 Status LED, P4 Power LED, U1 INA 169, U2 DC-DC_Stepdown, U3 MC33926, U4 ARDUINO_NANO

Commit message: sender_v2_geschlossen
3D Ansichten akktualisiert
Namen von Footprints umgeändet und angepasst an den neuen Bezeichnungen
von Kicad
----- keine Änderungen an Schaltplan vorgenommen -----
Parts:
- C1, C2: symbol CP1 -> CP1-RESCUE-Perimeter_sender_v2
- R1, R2, R3, R4, R5, R6, R7: symbol R -> R-RESCUE-Perimeter_sender_v2
- RV1, RV2: symbol POT -> POT-RESCUE-Perimeter_sender_v2
Changed lines of the file:
@@
 EESchema Schematic File Version 2
+LIBS:Perimeter sender v2-rescue
 LIBS:arduino_shieldsNCL
 LIBS:power
@@
 LIBS:memory
 LIBS:xilinx
-LIBS:special
 LIBS:microcontrollers
 LIBS:dsp
@@
 LIBS:ardumower mega shield svn-cache
 LIBS:Ina169
-EELAYER 25 0
+EELAYER 26 0
 EELAYER END
 $Descr A4 11693 8268
@@
 $EndComp
 $Comp
-L GND #PWR01
+L GND-RESCUE-Perimeter_sender_v2 #PWR01
 U 1 1 53A981F2
 P 10480 2170
@@
 $EndComp
 $Comp
-L GND #PWR02
+L GND-RESCUE-Perimeter_sender_v2 #PWR02
 U 1 1 53A98276
 P 8605 2945
@@
 M1_DuoLED_Schleife1_Rot
 $Comp
-L R R7
+L R-RESCUE-Perimeter_sender_v2 R7
 U 1 1 53A992CD
 P 6790 4750
@@
 $EndComp
 $Comp
-L R R5
+L R-RESCUE-Perimeter_sender_v2 R5
 U 1 1 53A992DC
 P 3550 5650
@@
 $EndComp
 $Comp
-L GND #PWR05
+L GND-RESCUE-Perimeter_sender_v2 #PWR05
 U 1 1 54D5004F
 P 1800 2275
@@
 $EndComp
 $Comp
-L GND #PWR06
+L GND-RESCUE-Perimeter_sender_v2 #PWR06
 U 1 1 54D500D0
 P 3150 3050
@@
 $EndComp
 $Comp
-L GND #PWR07
+L GND-RESCUE-Perimeter_sender_v2 #PWR07
 U 1 1 54D50107
 P 2300 3050
@@
 $EndComp
 $Comp
-L GND #PWR010
+L GND-RESCUE-Perimeter_sender_v2 #PWR010
 U 1 1 54D50837
 P 3675 6150
@@
 $EndComp
 $Comp
-L GND #PWR011
+L GND-RESCUE-Perimeter_sender_v2 #PWR011
 U 1 1 54D518BB
 P 2000 4125
@@
 $EndComp
 $Comp
-L GND #PWR012
+L GND-RESCUE-Perimeter_sender_v2 #PWR012
 U 1 1 54D51A61
 P 2600 3925
@@
 INA169
 $Comp
-L POT RV1
+L POT-RESCUE-Perimeter_sender_v2 RV1
 U 1 1 54D524A0
 P 1025 1025
@@
 $EndComp
 $Comp
-L GND #PWR014
+L GND-RESCUE-Perimeter_sender_v2 #PWR014
 U 1 1 54D527F0
 P 1125 1275
@@
 $EndComp
 $Comp
-L R R6
+L R-RESCUE-Perimeter_sender_v2 R6
 U 1 1 54D53F97
 P 3150 5550
@@
 $EndComp
 $Comp
-L R R4
+L R-RESCUE-Perimeter_sender_v2 R4
 U 1 1 54D5424D
 P 3550 5450
@@
 $EndComp
 $Comp
-L R R3
+L R-RESCUE-Perimeter_sender_v2 R3
 U 1 1 54D5428C
 P 3450 4750
@@
 $EndComp
 $Comp
-L CP1 C2
+L CP1-RESCUE-Perimeter_sender_v2 C2
 U 1 1 54D55373
 P 2625 1675
@@
 $EndComp
 $Comp
-L CP1 C1
+L CP1-RESCUE-Perimeter_sender_v2 C1
 U 1 1 54D555BA
 P 2250 1675
@@
 $EndComp
 $Comp
-L GND #PWR016
+L GND-RESCUE-Perimeter_sender_v2 #PWR016
 U 1 1 54D55677
 P 2625 1975
@@
 $EndComp
 $Comp
-L GND #PWR017
+L GND-RESCUE-Perimeter_sender_v2 #PWR017
 U 1 1 54D55697
 P 2250 1975
@@
 $EndComp
 $Comp
-L GND #PWR020
+L GND-RESCUE-Perimeter_sender_v2 #PWR020
 U 1 1 54D55FF9
 P 8655 1545
@@
 M2_DuoLED_Schleife2_Rot
 $Comp
-L R R1
+L R-RESCUE-Perimeter_sender_v2 R1
 U 1 1 54D586F5
 P 3150 1675
@@
 $EndComp
 $Comp
-L R R2
+L R-RESCUE-Perimeter_sender_v2 R2
 U 1 1 54D588A5
 P 3350 1675
@@
 LED_12V
 $Comp
-L GND #PWR024
+L GND-RESCUE-Perimeter_sender_v2 #PWR024
 U 1 1 54D58D55
 P 6575 2270
@@
 $EndComp
 $Comp
-L GND #PWR025
+L GND-RESCUE-Perimeter_sender_v2 #PWR025
 U 1 1 54F4DA22
 P 6755 980
@@
 $EndComp
 $Comp
-L GND #PWR026
+L GND-RESCUE-Perimeter_sender_v2 #PWR026
 U 1 1 54F4DB09
 P 6755 1180
@@
 $EndComp
 $Comp
-L GND #PWR027
+L GND-RESCUE-Perimeter_sender_v2 #PWR027
 U 1 1 54F4DB80
 P 6755 1480
@@
 $EndComp
 $Comp
-L GND #PWR028
+L GND-RESCUE-Perimeter_sender_v2 #PWR028
 U 1 1 54F4EA91
 P 6575 2070
@@
 $EndComp
 $Comp
-L GND #PWR029
+L GND-RESCUE-Perimeter_sender_v2 #PWR029
 U 1 1 54F74294
 P 8655 2445
@@
 NoConn ~ 5780 4950
 $Comp
-L POT RV2
+L POT-RESCUE-Perimeter_sender_v2 RV2
 U 1 1 54FCCD61
 P 1025 1695
@@
 $EndComp
 $Comp
-L GND #PWR030
+L GND-RESCUE-Perimeter_sender_v2 #PWR030
 U 1 1 54FCCD67
 P 1125 1945
