File: pcb/Produzierte_Platinen/sender_v2_geschlossen/Perimeter sender v2.kicad_pcb (KiCad board)
At the start: 2 copper layers, 110 x 59.9 mm, 27 parts, among them P1 Vin 24V, P2 VOut 24V, P3 Status LED, P4 Power LED, U1 INA 169, U2 DC-DC_Stepdown, U3 MC33926, U4 ARDUINO_NANO

Commit message: sender_v2_geschlossen
3D Ansichten akktualisiert
Namen von Footprints umgeändet und angepasst an den neuen Bezeichnungen
von Kicad
----- keine Änderungen an Schaltplan vorgenommen -----
Parts:
- U3: footprint sender_v2:MC_33926_31polig_mit_Bohrloch_neue_Masse -> Zimprich:MC_33926_31polig_mit_Bohrloch_neue_Masse

Commit message: sender_v2_geschlossen
sender_v2_geschlossen
Footprints und Libs angepasst an neue Kicad Version.
Dateiänderungen angepasst an neue Kicad Version.
Parts:
- B1, B2, B3, B5, B6: footprint sender_v2:Bohrloch_3,2mm -> Zimprich:Bohrloch_3,2mm
- C1, C2: footprint sender_v2:Elko_vert_11.2x6.3mm_RM2.5_RM5.0 -> Zimprich:Elko_vert_11.2x6.3mm_RM2.5_RM5.0
- D1: footprint sender_v2:MBR1045_Horizontal -> Zimprich:MBR1045_Horizontal
- EF1: footprint sender_v2:Fuseholder_Reichelt_PL112000 -> Zimprich:Fuseholder_Reichelt_PL112000
- JP1: footprint sender_v2:Pin_Header_Straight_1x02 -> Zimprich:Pin_Header_Straight_1x02
- P1, P2: footprint sender_v2:Anschlussklemme_2P_RM5,08 -> Zimprich:Anschlussklemme_2P_RM5,08
- P3: footprint Pin_Headers:Pin_Header_Straight_1x08 -> Connector_PinHeader_2.54mm:PinHeader_1x08_P2.54mm_Vertical
- P4: footprint Pin_Headers:Pin_Header_Straight_1x04 -> Connector_PinHeader_2.54mm:PinHeader_1x04_P2.54mm_Vertical
- R1, R2, R3, R4, R5, R6, R7: footprint sender_v2:Resistor_Horizontal_RM10mm -> Zimprich:Resistor_Horizontal_RM10mm
- RV1, RV2: footprint sender_v2:Potentiometer_VishaySpectrol-Econtrim-Type36T_3D-angepasst_Ardumover_Shop -> Zimprich:Potentiometer_VishaySpectrol-Econtrim-Type36T_3D-angepasst_Ardumover_Shop
- U1: footprint sender_v2:INA169 -> Zimprich:INA169
- U2: footprint sender_v2:DC_DC_DSN2596_mit_Bohrloch -> Zimprich:DC_DC_DSN2596_mit_Bohrloch
- U4: footprint sender_v2:arduino_nano -> Zimprich:arduino_nano
- moved B2 3.43 mm to (209.0, 115.2)
- moved B3 3.43 mm to (259.1, 115.2)
Connections:
- B1 pad 1: (no net) -> unconnected-(B1-Pad1)
- B2 pad 1: (no net) -> unconnected-(B2-Pad1)
- B3 pad 1: (no net) -> unconnected-(B3-Pad1)
- B5 pad 1: (no net) -> unconnected-(B5-Pad1)
- B6 pad 1: (no net) -> unconnected-(B6-Pad1)
- EF1 pad 1: Net-(D1-Pad1) -> Net-(D1-Pad2)
- U1 pad 4: Net-(D1-Pad1) -> Net-(D1-Pad2)
- U2 pad 3: Net-(D1-Pad2) -> Net-(D1-Pad1)
- U3 pad 1: (no net) -> unconnected-(U3-Pad1)
- U3 pad 11: (no net) -> unconnected-(U3-Pad11)
- U3 pad 12: (no net) -> unconnected-(U3-Pad12)
- U3 pad 19: (no net) -> unconnected-(U3-Pad19)
- U3 pad 20: (no net) -> unconnected-(U3-Pad20)
- U3 pad 23: (no net) -> unconnected-(U3-Pad23)
- U3 pad 24: (no net) -> unconnected-(U3-Pad24)
- U4 pad 3V3: (no net) -> unconnected-(U4-Pad3V3)
- U4 pad D10: (no net) -> unconnected-(U4-PadD10)
- U4 pad GND0: (no net) -> unconnected-(U4-PadGND0)
- U4 pad REF: (no net) -> unconnected-(U4-PadREF)
- U4 pad RST0: (no net) -> unconnected-(U4-PadRST0)
- U4 pad RST1: (no net) -> unconnected-(U4-PadRST1)
- U4 pad RX0: (no net) -> unconnected-(U4-PadRX0)
- U4 pad TX1: (no net) -> unconnected-(U4-PadTX1)
Routing:
- net Net-(D1-Pad2): track 41.1 -> 40.0 mm
- net Net-(D1-Pad1): track 40.0 -> 41.1 mm
- net POTI2: vias 2 -> 1
- net Net-(R7-Pad2): vias 2 -> 1
- net M2nD2 pwm: vias 2 -> 0
- net M1IN1: vias 2 -> 0
Other:
- net class Default removed
