File: pcb/Test_und_Entwicklung/Sunray_Platinen_Entwicklung_V3 _Serie/ArduSensorDuino_V3.00.ASD_geschlossen/ArduSensorDuino.sch (KiCad schematic (older format))
At the start: 106 parts, among them IC1 ATMEGA328-P, P1 DS18B20, P10 ICSP, P11 TWI, P12 VIN_, P13 RS232-TTL, P14 START/STOP, P15 ZONE OC, P16 SENSOR-OC, P17 USB-LIGHT, P2 SR04-1, P3 GP2Y-1, P4 SERVO, P5 VIN, P6 SR04-2, P7 GP2Y-2, P8 SR04-3, P9 GP2Y-3, Q1 16MHz, SW1 Reset, T1 BC847B, T2 BC847B, T3 BC847B, T4 BC847B, T5 BC847B, T6 BC847B, U1 LM2940CS-5.0, U2 LM2940CS-5.0

Commit message: ArduSensorDuino_V3.00.ASD_geschlossen
3D Ansichten aktualisiert
Namen von Footprints umgeändert und angepasst an die neuen Bezeichnungen
von Kicad
----- keine Änderungen am Schaltplan vorgenommen -----
Parts:
- LED1, LED2, LED3, LED4, LED5, LED6, LED7, LED8, LED9: symbol LED -> LED-RESCUE-ArduSensorDuino
Changed lines of the file:
@@
 EESchema Schematic File Version 2
+LIBS:ArduSensorDuino-rescue
 LIBS:power
 LIBS:device
@@
 LIBS:contrib
 LIBS:valves
-LIBS:MPX5010
-LIBS:OPA2340PA
-LIBS:LM2940CS-5.0
 LIBS:Zimprich
-EELAYER 25 0
+LIBS:ArduSensorDuino-cache
+EELAYER 26 0
 EELAYER END
 $Descr A4 11693 8268
@@
 $EndComp
 $Comp
-L LED LED1
+L LED-RESCUE-ArduSensorDuino LED1
 U 1 1 55CBC631
 P 3250 2800
@@
 $EndComp
 $Comp
-L LED LED2
+L LED-RESCUE-ArduSensorDuino LED2
 U 1 1 55CBC7ED
 P 3250 3150
@@
 $EndComp
 $Comp
-L LED LED3
+L LED-RESCUE-ArduSensorDuino LED3
 U 1 1 55CBC954
 P 3250 3550
@@
 $EndComp
 $Comp
-L LED LED5
+L LED-RESCUE-ArduSensorDuino LED5
 U 1 1 55CE3F68
 P 6100 1350
@@
 $EndComp
 $Comp
-L LED LED6
+L LED-RESCUE-ArduSensorDuino LED6
 U 1 1 5725DA8E
 P 5200 2800
@@
 $EndComp
 $Comp
-L LED LED7
+L LED-RESCUE-ArduSensorDuino LED7
 U 1 1 5725DC67
 P 5200 3200
@@
 $EndComp
 $Comp
-L LED LED8
+L LED-RESCUE-ArduSensorDuino LED8
 U 1 1 57291CA2
 P 5200 3600
@@
 $EndComp
 $Comp
-L LED LED9
+L LED-RESCUE-ArduSensorDuino LED9
 U 1 1 57291DD5
 P 5200 3950
@@
 +5V-SERVO
 $Comp
-L LED LED4
+L LED-RESCUE-ArduSensorDuino LED4
 U 1 1 57293B44
 P 5950 2150
@@
 00 00 80 0A 67 18 DC F4 02 28 33 BE 86 00 00 00 50 E1 68 F7 06 50 76 E4 DE 00 00 00 A8 7C 8C F7
 06 50 5E E4 DE 00 00 00 A8 70 59 D6 F7 2E 41 B8 61 8B 05 E0 5A F1 FF 3D 02 7B 6A FA 68 F9 99 00
-00 00 00 49 45 4E 44 AE 42 60 82 92
+00 00 00 49 45 4E 44 AE 42 60 82
 EndData
 $EndBitmap
