File: pcb/Test_und_Entwicklung/Sunray_Platinen_Entwicklung_V3 _Serie/ArduBumperPerimeterDuino_V3.00.ABPD_geschlossen/BumperDuino.kicad_pcb (KiCad board)
At the start: 2 copper layers, 96.5 x 66 mm, 71 parts, among them IC1 ATMEGA328-P, J4 J4, P1 Gy-521, Q1 16MHz, SW1 Reset, T1 BC847B, T2 BC847B, U1 MPX5010, U2 MPX5010, U4 OPA2340PA, U6 LM2940CS-5.0

Commit message: ArduBumperPerimeterDuino_V3.00.ABPD_geschlossen
ArduBumperPerimeterDuino_V3.00.ABPD_geschlossen
Symbole in der 3d Ansicht berichtigt wegen neuer KIcad Symbol Ansichten
RoHS Symbol und Mülleimer Symbol hinzugefügt
------------------------------------------------------------------------
Es wurden keine Änderungen am Schaltplan,Layout oder dergleichen
vorgenommen
------------------------------------------------------------------------
Parts:
- added REF***: WEEE-Logo_4.2x6mm_SilkScreen, Symbols:WEEE-Logo_4.2x6mm_SilkScreen, F.Cu at (66.3, 94.4)
Other:
- net class Default: clearance 0.2 -> 0
- rule trace_clearance: 0.2 -> 0
- board text added: "RoHS"
