File: pcb/Test_und_Entwicklung/Sunray_Platinen_Entwicklung_V3 _Serie/ArduBumperPerimeterDuino_V3.00.ABPD_geschlossen/BumperDuino.sch (KiCad schematic (older format))
At the start: 71 parts, among them IC1 ATMEGA328-P, J4 J4, P1 Gy-521, Q1 16MHz, SW1 Reset, T1 BC847B, T2 BC847B, U1 MPX5010, U2 MPX5010, U4 OPA2340PA, U6 LM2940CS-5.0

Commit message: ArduBumperPerimeterDuino_V3.00.ABPD_geschlossen
ArduBumperPerimeterDuino_V3.00.ABPD_geschlossen
Symbole in der 3d Ansicht berichtigt wegen neuer KIcad Symbol Ansichten
RoHS Symbol und Mülleimer Symbol hinzugefügt
------------------------------------------------------------------------
Es wurden keine Änderungen am Schaltplan,Layout oder dergleichen
vorgenommen
------------------------------------------------------------------------
Parts:
- ACTIVE1, Fault1, OK1, PowerOK1, Sensor1, Sensor2: symbol LED -> LED-RESCUE-BumperDuino
- U2: Bauform (none) -> Value; Bestelllink (none) -> Value; Bestellnummer (none) -> Value; Funktion (none) -> Value; Gehäuseart (none) -> Value; Hersteller (none) -> Value; Hersteller Bestellnummer (none) -> Value; Technische Daten (none) -> Value
Changed lines of the file:
@@
 EESchema Schematic File Version 2
+LIBS:BumperDuino-rescue
 LIBS:power
 LIBS:device
@@
 LIBS:adc-dac
 LIBS:memory
-LIBS:xilinx
 LIBS:microcontrollers
 LIBS:dsp
@@
 LIBS:contrib
 LIBS:valves
-LIBS:MPX5010
-LIBS:OPA2340PA
-LIBS:LM2940CS-5.0
 LIBS:Zimprich
 LIBS:BumperDuino-cache
-EELAYER 25 0
+EELAYER 26 0
 EELAYER END
 $Descr A4 11693 8268
@@
 $EndComp
 $Comp
-L LED ACTIVE1
+L LED-RESCUE-BumperDuino ACTIVE1
 U 1 1 55CBC631
 P 2900 1850
@@
 $EndComp
 $Comp
-L LED Sensor2
+L LED-RESCUE-BumperDuino Sensor2
 U 1 1 55CBC7ED
 P 2900 2200
@@
 $EndComp
 $Comp
-L LED Sensor1
+L LED-RESCUE-BumperDuino Sensor1
 U 1 1 55CBC954
 P 2900 2600
@@
 $EndComp
 $Comp
-L LED PowerOK1
+L LED-RESCUE-BumperDuino PowerOK1
 U 1 1 55CE3F68
 P 4700 1750
@@
 F 2 "MPX5010:867C-H" H 7050 3350 60  0001 C CNN
 F 3 "" H 7050 3350 60  0000 C CNN
+F 4 "Value" H 7050 3350 60  0001 C CNN "Gehäuseart"
+F 5 "Value" H 7050 3350 60  0001 C CNN "Bestelllink"
+F 6 "Value" H 7050 3350 60  0001 C CNN "Technische Daten"
+F 7 "Value" H 7050 3350 60  0001 C CNN "Bestellnummer"
+F 8 "Value" H 7050 3350 60  0001 C CNN "Bauform"
+F 9 "Value" H 7050 3350 60  0001 C CNN "Funktion"
+F 10 "Value" H 7050 3350 60  0001 C CNN "Hersteller"
+F 11 "Value" H 7050 3350 60  0001 C CNN "Hersteller Bestellnummer"
 	1    7050 3350
 	1    0    0    -1
@@
 F9 0E 00 00 00 00 00 C0 F9 46 BE 03 00 00 00 00 00 70 BE 91 EF 00 00 00 00 00 00 9C 6F E4 3B 00
 00 00 00 00 00 E7 1B F9 0E 00 00 00 00 00 C0 F9 F6 FF 01 5A 01 1C DD 8D 3A 8E 97 00 00 00 00 49
-45 4E 44 AE 42 60 82 FF
+45 4E 44 AE 42 60 82
 EndData
 $EndBitmap
@@
 LED-INIT-OK
 $Comp
-L LED Fault1
+L LED-RESCUE-BumperDuino Fault1
 U 1 1 5725DA8E
 P 2900 3050
@@
 $EndComp
 $Comp
-L LED OK1
+L LED-RESCUE-BumperDuino OK1
 U 1 1 5725DC67
 P 2900 3450
@@
 Wire Wire Line
 	8850 5700 8850 6000
-Text Notes 11770 4905 0    60   ~ 0
+Text Notes 8755 1110 0    60   ~ 0
 21.05.2016\nDiode D1 pad von 0,7 auf 1,016 vergrößert\nvon T1 und T2 lib ausgetauscht
 $Comp
