File: pcb/Test_und_Entwicklung/ArduMower_RaspberryPi_Power_Switch_V1.0_geoeffnet/ArduMower_RaspberryPi_Power_Switch.sch (KiCad schematic (older format))
At the start: 128 parts, among them IC1 74ALS05N, IC2 74LS73N, J1 TWI EXTERN 5V, J2 CONN_01X02, J3 CONN_01X02, J4 CONN_01X02, J5 CONN_01X02, J6 CONN_01X10, J7 DHT22 3,3V, K1 APF30212C, K2 APF30212C, K3 APF30212C, Q1 NDB6020P, Q2 IRF 9540NS, Q3 BC817, Q4 BC817, Q5 BC817, Q6 BC817, SW1 Tact_Switch_12x12mm_with_inte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, SW2 Reset, U1 PCA9517D, U2 PCA9517D

Commit message: ArduMower_RaspberryPi_Power_Switch_V1.0_geoeffnet
ArduMower_RaspberryPi_Power_Switch_V1.0_geoeffnet
Widerstand R37 hinzugefügt
Durchkontaktierung bei R16 verschoben
Beschriftungen angeordnet
Parts:
- added R37: 2K2, Resistors_SMD:R_1206, symbol R
- Q3: Bestelllink Value -> https://www.reichelt.de/index.html?ACTION=446&LA=3
Connections:
- net GND: now also R37.1
- net N$11: now also R37.2
Changed lines of the file:
@@
 F 3 "" H 3570 6970 50  0000 L CNN
 F 4 "Value" H 3570 6970 60  0001 C CNN "Gehäuseart"
-F 5 "Value" H 3570 6970 60  0001 C CNN "Bestelllink"
+F 5 "https://www.reichelt.de/index.html?ACTION=446&LA=3" H 3570 6970 60  0001 C CNN "Bestelllink"
 F 6 "Value" H 3570 6970 60  0001 C CNN "Technische Daten"
 F 7 "Value" H 3570 6970 60  0001 C CNN "Bestellnummer"
@@
 Text Notes 1060 6770 0    60   ~ 0
 Hinzugefügt
+$Comp
+L R R37
+U 1 1 58A6DCA1
+P 7260 5560
+F 0 "R37" H 7340 5575 50  0000 L CNN
+F 1 "2K2" H 7340 5490 50  0000 L CNN
+F 2 "Resistors_SMD:R_1206" H 7348 5469 50  0001 L CNN
+F 3 "" H 7260 5560 50  0000 C CNN
+F 4 "Value" H 7260 5560 60  0001 C CNN "Gehäuseart"
+F 5 "Value" H 7260 5560 60  0001 C CNN "Bestelllink"
+F 6 "Value" H 7260 5560 60  0001 C CNN "Technische Daten"
+F 7 "Value" H 7260 5560 60  0001 C CNN "Bestellnummer"
+F 8 "Value" H 7260 5560 60  0001 C CNN "Bauform"
+F 9 "Value" H 7348 5423 60  0001 L CNN "Funktion"
+F 10 "Value" H 7260 5560 60  0001 C CNN "Hersteller"
+F 11 "Value" H 7260 5560 60  0001 C CNN "Hersteller Bestellnummer"
+	1    7260 5560
+	-1   0    0    1
+$EndComp
+Wire Wire Line
+	7260 5710 7260 5870
+$Comp
+L GND #PWR066
+U 1 1 58A6ED16
+P 7260 5870
+F 0 "#PWR066" H 7260 5620 50  0001 C CNN
+F 1 "GND" H 7265 5697 50  0000 C CNN
+F 2 "" H 7260 5870 50  0000 C CNN
+F 3 "" H 7260 5870 50  0000 C CNN
+	1    7260 5870
+	1    0    0    -1
+$EndComp
+Wire Wire Line
+	7260 5410 7260 5270
+Connection ~ 7260 5270
 $EndSCHEMATC

Commit message: ArduMower_RaspberryPi_Power_Switch_V1.0_geoeffnet
ArduMower_RaspberryPi_Power_Switch_V1.0_geoeffnet
RoHos Beschriftung und Mülleimer hinzugefügt
Parts:
- Q1, Q2: symbol IRF9540N -> IRF9540N-RESCUE-ArduMower_RaspberryPi_Power_Switch
Changed lines of the file:
@@
 EESchema Schematic File Version 2
+LIBS:ArduMower_RaspberryPi_Power_Switch-rescue
 LIBS:diode
 LIBS:transistors
@@
 SCLPI
 $Comp
-L IRF9540N Q2
+L IRF9540N-RESCUE-ArduMower_RaspberryPi_Power_Switch Q2
 U 1 1 585F12A5
 P 3520 8470
@@
 $EndComp
 $Comp
-L IRF9540N Q1
+L IRF9540N-RESCUE-ArduMower_RaspberryPi_Power_Switch Q1
 U 1 1 585F4557
 P 7720 8820
