File: pcb/Produzierte_Platinen/megashield_svn_1.3_geschlossen/LShifter1.sch (KiCad schematic (older format))
At the start: 3 parts, among them Q5 BSS138

Commit message: megashield_svn_1.3_geschlossen
megashield_svn_1.3_geschlossen
Schönheitsfehler in Plan verbessert
Bei dem globalen Maker "pinRemoteSwitch" war in den Schaltpanseite bei
dem Due die Signalrichtung falsch eingezeichnet.
Signalrichtung wurde  umgeändert
Die Änderung hat kein Einfluß auf die Funktion der Schaltung
Parts:
- Q5: symbol BSS138-RESCUE-ardumower_mega_shield_svn -> ardumower-mega-shield-svn-rescue:BSS138-RESCUE-ardumower_mega_shield_svn
- R58, R59: symbol R -> ardumower-mega-shield-svn-rescue:R-RESCUE-ardumower_mega_shield_svn
Changed lines of the file:
@@
-EESchema Schematic File Version 2
-LIBS:ardumower mega shield svn-rescue
-LIBS:power
-LIBS:device
-LIBS:Zimprich
-LIBS:conn
-LIBS:transistors
-LIBS:switches
-LIBS:linear
-LIBS:texas
-LIBS:diode
+EESchema Schematic File Version 4
 LIBS:ardumower mega shield svn-cache
 EELAYER 26 0
@@
 	5210 3735 5605 3735
 $Comp
-L R R59
+L ardumower-mega-shield-svn-rescue:R-RESCUE-ardumower_mega_shield_svn R59
 U 1 1 57E6FCAE
 P 6110 3250
@@
 $EndComp
 $Comp
-L R R58
+L ardumower-mega-shield-svn-rescue:R-RESCUE-ardumower_mega_shield_svn R58
 U 1 1 57E6FCB7
 P 5435 3250
@@
 IOREF
 $Comp
-L BSS138-RESCUE-ardumower_mega_shield_svn Q5
+L ardumower-mega-shield-svn-rescue:BSS138-RESCUE-ardumower_mega_shield_svn Q5
 U 1 1 57EB0392
 P 5805 3635
@@
 $EndComp
 $Comp
-L +5VP #PWR0131
+L ardumower-mega-shield-svn-rescue:+5VP-RESCUE-ardumower_mega_shield_svn #PWR0131
 U 1 1 57FA7DCF
 P 6110 2900
