File: pcb/Produzierte_Platinen/megashield_svn_1.3_geschlossen/Leuchtdioden.sch (KiCad schematic (older format))
At the start: 47 parts, among them IC1 UDN 2987 LWTR-6T, P10 Status LEDs GND, P50 Led Panel, P7 Status LEDs, Q14 BC817, Q15 BC817, Q16 BC817, Q17 BC817, Q18 BC817, Q19 BC817, Q20 BC817, Q21 BC817, Q22 BC817, Q23 BC817

Commit message: megashield_svn_1.3_geschlossen
megashield_svn_1.3_geschlossen
Schönheitsfehler in Plan verbessert
Bei dem globalen Maker "pinRemoteSwitch" war in den Schaltpanseite bei
dem Due die Signalrichtung falsch eingezeichnet.
Signalrichtung wurde  umgeändert
Die Änderung hat kein Einfluß auf die Funktion der Schaltung
Parts:
- C18: symbol C_Small -> ardumower-mega-shield-svn-rescue:C_Small-RESCUE-ardumower_mega_shield_svn
- D17, D18, D19, D20, D21, D22, D23: symbol LED_Small -> ardumower-mega-shield-svn-rescue:LED_Small-RESCUE-ardumower_mega_shield_svn
- IC1: symbol UDN2987A-6-T -> ardumower-mega-shield-svn-rescue:UDN2987A-6-T-RESCUE-ardumower_mega_shield_svn
- P10: symbol CONN_01X10 -> ardumower-mega-shield-svn-rescue:CONN_01X10-RESCUE-ardumower_mega_shield_svn
- P50: symbol CONN_02X07 -> ardumower-mega-shield-svn-rescue:CONN_02X07-RESCUE-ardumower_mega_shield_svn
- P7: symbol CONN_01X14 -> ardumower-mega-shield-svn-rescue:CONN_01X14-RESCUE-ardumower_mega_shield_svn
- Q14, Q15, Q16, Q17, Q18, Q19, Q20, Q21, Q22, Q23: symbol BC817-40 -> ardumower-mega-shield-svn-rescue:BC817-40-RESCUE-ardumower_mega_shield_svn
- R1, R11, R134, R17, R19, R2, R20, R21, R22, R23, R24, R25, R38, R43, R5, R74, R75, R76, R77, R78, R79, R80, R81: symbol R -> ardumower-mega-shield-svn-rescue:R-RESCUE-ardumower_mega_shield_svn
- SP1, SP2: symbol SPEAKER -> ardumower-mega-shield-svn-rescue:SPEAKER-RESCUE-ardumower_mega_shield_svn
