File: pcb/Produzierte_Platinen/megashield_svn_1.3_geschlossen/Motortreiber.sch (KiCad schematic (older format))
At the start: 8 parts, among them P15 Left, P18 Right, P36 Res24V-2, P37 Mower, P39 Res24V-1

Commit message: megashield_svn_1.3_geschlossen
megashield_svn_1.3_geschlossen
Schönheitsfehler in Plan verbessert
Bei dem globalen Maker "pinRemoteSwitch" war in den Schaltpanseite bei
dem Due die Signalrichtung falsch eingezeichnet.
Signalrichtung wurde  umgeändert
Die Änderung hat kein Einfluß auf die Funktion der Schaltung
Parts:
- Dual1, Dual2: symbol MC33926 -> ardumower-mega-shield-svn-rescue:MC33926-RESCUE-ardumower_mega_shield_svn
- JP3: symbol Jumper -> ardumower-mega-shield-svn-rescue:Jumper-RESCUE-ardumower_mega_shield_svn
- P15, P18, P36, P37, P39: symbol CONN_01X02 -> ardumower-mega-shield-svn-rescue:CONN_01X02-RESCUE-ardumower_mega_shield_svn
Changed lines of the file:
@@
-EESchema Schematic File Version 2
-LIBS:ardumower mega shield svn-rescue
-LIBS:power
-LIBS:device
-LIBS:Zimprich
-LIBS:conn
-LIBS:transistors
-LIBS:switches
-LIBS:linear
-LIBS:texas
-LIBS:diode
+EESchema Schematic File Version 4
 LIBS:ardumower mega shield svn-cache
 EELAYER 26 0
@@
 $EndDescr
 $Comp
-L MC33926 Dual1
+L ardumower-mega-shield-svn-rescue:MC33926-RESCUE-ardumower_mega_shield_svn Dual1
 U 1 1 57D96B1D
 P 4510 2375
@@
 pinMotorRightFault
 $Comp
-L MC33926 Dual2
+L ardumower-mega-shield-svn-rescue:MC33926-RESCUE-ardumower_mega_shield_svn Dual2
 U 1 1 57D96B33
 P 4510 5025
@@
 ReserveAD6
 $Comp
-L Jumper JP3
+L ardumower-mega-shield-svn-rescue:Jumper-RESCUE-ardumower_mega_shield_svn JP3
 U 1 1 57D96C22
 P 2795 4975
@@
 	2495 4975 2425 4975
 $Comp
-L GND #PWR013
+L ardumower-mega-shield-svn-rescue:GND-RESCUE-ardumower_mega_shield_svn #PWR013
 U 1 1 57DCB31A
 P 7305 2190
@@
 $EndComp
 $Comp
-L GND #PWR014
+L ardumower-mega-shield-svn-rescue:GND-RESCUE-ardumower_mega_shield_svn #PWR014
 U 1 1 57DCB496
 P 3510 3025
@@
 $EndComp
 $Comp
-L GND #PWR015
+L ardumower-mega-shield-svn-rescue:GND-RESCUE-ardumower_mega_shield_svn #PWR015
 U 1 1 57DCB679
 P 3510 2525
@@
 $EndComp
 $Comp
-L GND #PWR016
+L ardumower-mega-shield-svn-rescue:GND-RESCUE-ardumower_mega_shield_svn #PWR016
 U 1 1 57DCB703
 P 3510 1625
@@
 $EndComp
 $Comp
-L GND #PWR017
+L ardumower-mega-shield-svn-rescue:GND-RESCUE-ardumower_mega_shield_svn #PWR017
 U 1 1 57DCB93A
 P 3510 4275
@@
 $EndComp
 $Comp
-L GND #PWR018
+L ardumower-mega-shield-svn-rescue:GND-RESCUE-ardumower_mega_shield_svn #PWR018
 U 1 1 57DCBAED
 P 3330 5175
@@
 $EndComp
 $Comp
-L GND #PWR019
+L ardumower-mega-shield-svn-rescue:GND-RESCUE-ardumower_mega_shield_svn #PWR019
 U 1 1 57DCBBA3
 P 3510 5675
@@
 	7600 4665 7735 4665
 $Comp
-L GND #PWR020
+L ardumower-mega-shield-svn-rescue:GND-RESCUE-ardumower_mega_shield_svn #PWR020
 U 1 1 57DC2092
 P 7735 4840
@@
 	5385 4725 5385 4675
 $Comp
-L GND #PWR021
+L ardumower-mega-shield-svn-rescue:GND-RESCUE-ardumower_mega_shield_svn #PWR021
 U 1 1 57DC50B6
 P 10310 1730
@@
 	10445 1730 10310 1730
 $Comp
-L GND #PWR022
+L ardumower-mega-shield-svn-rescue:GND-RESCUE-ardumower_mega_shield_svn #PWR022
 U 1 1 57DC5B70
 P 10315 1095
@@
 	10450 1095 10315 1095
 $Comp
-L CONN_01X02 P39
+L ardumower-mega-shield-svn-rescue:CONN_01X02-RESCUE-ardumower_mega_shield_svn P39
 U 1 1 57E0418F
 P 10645 1680
@@
 $EndComp
 $Comp
-L CONN_01X02 P36
+L ardumower-mega-shield-svn-rescue:CONN_01X02-RESCUE-ardumower_mega_shield_svn P36
 U 1 1 57E067EC
 P 10650 1045
@@
 $EndComp
 $Comp
-L CONN_01X02 P37
+L ardumower-mega-shield-svn-rescue:CONN_01X02-RESCUE-ardumower_mega_shield_svn P37
 U 1 1 57E0AFDE
 P 7555 4175
@@
 	7255 4125 7355 4125
 $Comp
-L CONN_01X02 P15
+L ardumower-mega-shield-svn-rescue:CONN_01X02-RESCUE-ardumower_mega_shield_svn P15
 U 1 1 57E0CA53
 P 7120 2755
@@
 	6860 2705 6920 2705
 $Comp
-L CONN_01X02 P18
+L ardumower-mega-shield-svn-rescue:CONN_01X02-RESCUE-ardumower_mega_shield_svn P18
 U 1 1 57E0DF43
 P 7140 1525
