File: pcb/Produzierte_Platinen/megashield_svn_1.3_geschlossen/Motortreiber1.sch (KiCad schematic (older format))
At the start: 3 parts

Commit message: megashield_svn_1.3_geschlossen
megashield_svn_1.3_geschlossen
Schönheitsfehler in Plan verbessert
Bei dem globalen Maker "pinRemoteSwitch" war in den Schaltpanseite bei
dem Due die Signalrichtung falsch eingezeichnet.
Signalrichtung wurde  umgeändert
Die Änderung hat kein Einfluß auf die Funktion der Schaltung
Parts:
- C10: symbol CP1 -> ardumower-mega-shield-svn-rescue:CP1-RESCUE-ardumower_mega_shield_svn
- DKE1: symbol D -> ardumower-mega-shield-svn-rescue:D-RESCUE-ardumower_mega_shield_svn
- PRFA1: symbol F_10A -> ardumower-mega-shield-svn-rescue:F_10A-RESCUE-ardumower_mega_shield_svn
Changed lines of the file:
@@
-EESchema Schematic File Version 2
-LIBS:ardumower mega shield svn-rescue
-LIBS:power
-LIBS:device
-LIBS:Zimprich
-LIBS:conn
-LIBS:transistors
-LIBS:switches
-LIBS:linear
-LIBS:texas
-LIBS:diode
+EESchema Schematic File Version 4
 LIBS:ardumower mega shield svn-cache
 EELAYER 26 0
@@
 Dual1_IN_GND
 $Comp
-L F_10A PRFA1
+L ardumower-mega-shield-svn-rescue:F_10A-RESCUE-ardumower_mega_shield_svn PRFA1
 U 1 1 57DB8844
 P 2990 3700
@@
 	4640 4120 4640 4290
 $Comp
-L CP1 C10
+L ardumower-mega-shield-svn-rescue:CP1-RESCUE-ardumower_mega_shield_svn C10
 U 1 1 57DB8845
 P 3325 3990
@@
 Connection ~ 3325 4290
 $Comp
-L D DKE1
+L ardumower-mega-shield-svn-rescue:D-RESCUE-ardumower_mega_shield_svn DKE1
 U 1 1 57DB8937
 P 4370 4005
