File: pcb/Produzierte_Platinen/megashield_svn_1.3_geschlossen/OdoTeiler.sch (KiCad schematic (older format))
At the start: 11 parts, among them U12 4017, U4 4017, U5 4081, U9 4017

Commit message: megashield_svn_1.3_geschlossen
megashield_svn_1.3_geschlossen
Schönheitsfehler in Plan verbessert
Bei dem globalen Maker "pinRemoteSwitch" war in den Schaltpanseite bei
dem Due die Signalrichtung falsch eingezeichnet.
Signalrichtung wurde  umgeändert
Die Änderung hat kein Einfluß auf die Funktion der Schaltung
Parts:
- C14, C15, C16, C17: symbol C_Small -> ardumower-mega-shield-svn-rescue:C_Small-RESCUE-ardumower_mega_shield_svn
- S1, S2, S3: symbol SW_DIP_x8 -> ardumower-mega-shield-svn-rescue:SW_DIP_x8-RESCUE-ardumower_mega_shield_svn
- U12, U4, U9: symbol 4017 -> ardumower-mega-shield-svn-rescue:4017-RESCUE-ardumower_mega_shield_svn
- U5: symbol 4081 -> ardumower-mega-shield-svn-rescue:4081-RESCUE-ardumower_mega_shield_svn
Changed lines of the file:
@@
-EESchema Schematic File Version 2
-LIBS:ardumower mega shield svn-rescue
-LIBS:power
-LIBS:device
-LIBS:Zimprich
-LIBS:conn
-LIBS:transistors
-LIBS:switches
-LIBS:linear
-LIBS:texas
-LIBS:diode
+EESchema Schematic File Version 4
 LIBS:ardumower mega shield svn-cache
 EELAYER 26 0
@@
 [22:56:35 | Bearbeitet 22:58:38] Jürgen Lange: @uwe hier der teiler kann noch verfeinert werden und du brauchst die mimik 2x also den 4017 x2 und ein und gatter vom 4081 zusätzlich damit sind dann noch zwei übrig die arbeiten dann als or durch die negative logik timing-probleme werden so vermieden und die signale sin im sync \n[22:59:19] Kurzschuss - Uwe: sekunde diese Schaltung also mal 4\n[23:00:01] Kurzschuss - Uwe: wir haben ja 4 Odemetrie Pins\n[23:00:34] Jürgen Lange: natürlich wie immer die 100nF block nicht vergessen und beachten hinten hast du 5v pegel da muss man also noch was machen............................. ne die schaltung eigentlich nur 2x oder 3 mal wenn du den mäh-motor auch so machen möchtest\n[23:01:44 | Bearbeitet 23:05:06] Jürgen Lange: wir brauchen nur einen pro motor oneway die richtung kann uns wurst sein und vergesse die pullup nicht am eingang die werden trotzdem gebraucht\n[23:01:52 | Bearbeitet 23:02:17] Kurzschuss - Uwe: Also werten wir bei der Odemetrie nicht mehr two way aus sondern nur noch One way?\n[23:02:43] Kurzschuss - Uwe: wir haben ja bei unseren Motoren vor und Rückwärsts\n[23:03:20] Jürgen Lange: das ist ein dekadenzähler schau dir das datenblatt an dann kommst du sicher drauf\n[23:03:47] Kurzschuss - Uwe: okay\n[23:04:16] Jürgen Lange: die richtung kommt von der software wozu sollen wir das auswerten alexander weiß doch wo er hinfährt sind nur unnötige ints\n[23:05:40] Kurzschuss - Uwe: Dann hätten wir wider 2Pins mehr frei :)\n[23:08:58] Kurzschuss - Uwe: braucht der 4017 keine ´5V
 $Comp
-L 4017 U4
+L ardumower-mega-shield-svn-rescue:4017-RESCUE-ardumower_mega_shield_svn U4
 U 1 1 57F328FB
 P 2260 2070
@@
 $EndComp
 $Comp
-L 4081 U5
+L ardumower-mega-shield-svn-rescue:4081-RESCUE-ardumower_mega_shield_svn U5
 U 1 1 57F32953
 P 4015 1145
@@
 $EndComp
 $Comp
-L 4081 U5
+L ardumower-mega-shield-svn-rescue:4081-RESCUE-ardumower_mega_shield_svn U5
 U 4 1 57F32B77
 P 8275 1170
@@
 NoConn ~ 2810 2570
 $Comp
-L GND #PWR0138
+L ardumower-mega-shield-svn-rescue:GND-RESCUE-ardumower_mega_shield_svn #PWR0138
 U 1 1 57F36BEA
 P 1645 1865
@@
 	1645 1770 1710 1770
 $Comp
-L GND #PWR0139
+L ardumower-mega-shield-svn-rescue:GND-RESCUE-ardumower_mega_shield_svn #PWR0139
 U 1 1 57F37705
 P 2260 2790
@@
 5V an pin 16 richtig?\npin 16 richtig?\noder 5VP an pin 16
 $Comp
-L GND #PWR0140
+L ardumower-mega-shield-svn-rescue:GND-RESCUE-ardumower_mega_shield_svn #PWR0140
 U 1 1 57F39A30
 P 7635 1465
@@
 Connection ~ 7635 1270
 $Comp
-L GND #PWR0141
+L ardumower-mega-shield-svn-rescue:GND-RESCUE-ardumower_mega_shield_svn #PWR0141
 U 1 1 57F3A684
 P 4015 1465
@@
 5V an pin 14 richtig?\npin 16 richtig?\noder 5VP an pin 16
 $Comp
-L SW_DIP_x8 S1
+L ardumower-mega-shield-svn-rescue:SW_DIP_x8-RESCUE-ardumower_mega_shield_svn S1
 U 1 1 57F3CE2A
 P 3240 2070
@@
 Ausgang2
 $Comp
-L 4017 U9
+L ardumower-mega-shield-svn-rescue:4017-RESCUE-ardumower_mega_shield_svn U9
 U 1 1 57F7E24A
 P 2045 5225
@@
 $EndComp
 $Comp
-L 4081 U5
+L ardumower-mega-shield-svn-rescue:4081-RESCUE-ardumower_mega_shield_svn U5
 U 2 1 57F7E250
 P 3800 4300
@@
 NoConn ~ 2595 5725
 $Comp
-L GND #PWR0142
+L ardumower-mega-shield-svn-rescue:GND-RESCUE-ardumower_mega_shield_svn #PWR0142
 U 1 1 57F7E260
 P 1430 5020
@@
 	1430 4925 1495 4925
 $Comp
-L GND #PWR0143
+L ardumower-mega-shield-svn-rescue:GND-RESCUE-ardumower_mega_shield_svn #PWR0143
 U 1 1 57F7E268
 P 2045 5945
@@
 5V an pin 14 richtig?\npin 16 richtig?\noder 5VP an pin 16
 $Comp
-L SW_DIP_x8 S2
+L ardumower-mega-shield-svn-rescue:SW_DIP_x8-RESCUE-ardumower_mega_shield_svn S2
 U 1 1 57F7E28A
 P 3025 5225
@@
 Ausgang3
 $Comp
-L 4017 U12
+L ardumower-mega-shield-svn-rescue:4017-RESCUE-ardumower_mega_shield_svn U12
 U 1 1 57F7E516
 P 7630 5085
@@
 $EndComp
 $Comp
-L 4081 U5
+L ardumower-mega-shield-svn-rescue:4081-RESCUE-ardumower_mega_shield_svn U5
 U 3 1 57F7E521
 P 9385 4160
@@
 NoConn ~ 8180 5585
 $Comp
-L GND #PWR0144
+L ardumower-mega-shield-svn-rescue:GND-RESCUE-ardumower_mega_shield_svn #PWR0144
 U 1 1 57F7E531
 P 7015 4880
@@
 	7015 4785 7080 4785
 $Comp
-L GND #PWR0145
+L ardumower-mega-shield-svn-rescue:GND-RESCUE-ardumower_mega_shield_svn #PWR0145
 U 1 1 57F7E539
 P 7630 5805
@@
 5V an pin 16 richtig?\npin 16 richtig?\noder 5VP an pin 16
 $Comp
-L SW_DIP_x8 S3
+L ardumower-mega-shield-svn-rescue:SW_DIP_x8-RESCUE-ardumower_mega_shield_svn S3
 U 1 1 57F7E55B
 P 8610 5085
@@
 	3680 1720 3540 1720
 $Comp
-L +5VP #PWR0146
+L ardumower-mega-shield-svn-rescue:+5VP-RESCUE-ardumower_mega_shield_svn #PWR0146
 U 1 1 57F9F288
 P 4015 850
@@
 $EndComp
 $Comp
-L +5VP #PWR0147
+L ardumower-mega-shield-svn-rescue:+5VP-RESCUE-ardumower_mega_shield_svn #PWR0147
 U 1 1 57F9F31C
 P 2260 1375
@@
 $EndComp
 $Comp
-L +5VP #PWR0148
+L ardumower-mega-shield-svn-rescue:+5VP-RESCUE-ardumower_mega_shield_svn #PWR0148
 U 1 1 57F9F52A
 P 2045 4530
@@
 $EndComp
 $Comp
-L +5VP #PWR0149
+L ardumower-mega-shield-svn-rescue:+5VP-RESCUE-ardumower_mega_shield_svn #PWR0149
 U 1 1 57F9F7C4
 P 7630 4390
@@
 $EndComp
 $Comp
-L C_Small C15
+L ardumower-mega-shield-svn-rescue:C_Small-RESCUE-ardumower_mega_shield_svn C15
 U 1 1 57FBF162
 P 7055 2585
@@
 $EndComp
 $Comp
-L +5VP #PWR0150
+L ardumower-mega-shield-svn-rescue:+5VP-RESCUE-ardumower_mega_shield_svn #PWR0150
 U 1 1 57FBF2AC
 P 7055 2455
@@
 	7055 2485 7055 2455
 $Comp
-L GND #PWR0151
+L ardumower-mega-shield-svn-rescue:GND-RESCUE-ardumower_mega_shield_svn #PWR0151
 U 1 1 57FBF786
 P 7055 2735
@@
 	7055 2735 7055 2685
 $Comp
-L C_Small C16
+L ardumower-mega-shield-svn-rescue:C_Small-RESCUE-ardumower_mega_shield_svn C16
 U 1 1 57FBFD57
 P 7515 2580
@@
 $EndComp
 $Comp
-L +5VP #PWR0152
+L ardumower-mega-shield-svn-rescue:+5VP-RESCUE-ardumower_mega_shield_svn #PWR0152
 U 1 1 57FBFD5D
 P 7515 2450
@@
 	7515 2480 7515 2450
 $Comp
-L GND #PWR0153
+L ardumower-mega-shield-svn-rescue:GND-RESCUE-ardumower_mega_shield_svn #PWR0153
 U 1 1 57FBFD64
 P 7515 2730
@@
 	7515 2730 7515 2680
 $Comp
-L C_Small C14
+L ardumower-mega-shield-svn-rescue:C_Small-RESCUE-ardumower_mega_shield_svn C14
 U 1 1 57FBFDB1
 P 6610 2595
@@
 $EndComp
 $Comp
-L +5VP #PWR0154
+L ardumower-mega-shield-svn-rescue:+5VP-RESCUE-ardumower_mega_shield_svn #PWR0154
 U 1 1 57FBFDB7
 P 6610 2465
@@
 	6610 2495 6610 2465
 $Comp
-L GND #PWR0155
+L ardumower-mega-shield-svn-rescue:GND-RESCUE-ardumower_mega_shield_svn #PWR0155
 U 1 1 57FBFDBE
 P 6610 2745
@@
 	6610 2745 6610 2695
 $Comp
-L C_Small C17
+L ardumower-mega-shield-svn-rescue:C_Small-RESCUE-ardumower_mega_shield_svn C17
 U 1 1 57FBFF07
 P 8010 2595
@@
 $EndComp
 $Comp
-L +5VP #PWR0156
+L ardumower-mega-shield-svn-rescue:+5VP-RESCUE-ardumower_mega_shield_svn #PWR0156
 U 1 1 57FBFF0D
 P 8010 2465
@@
 	8010 2495 8010 2465
 $Comp
-L GND #PWR0157
+L ardumower-mega-shield-svn-rescue:GND-RESCUE-ardumower_mega_shield_svn #PWR0157
 U 1 1 57FBFF14
 P 8010 2745
