File: pcb/Produzierte_Platinen/megashield_svn_1.3_geschlossen/Spannungsversorgung.sch (KiCad schematic (older format))
At the start: 21 parts, among them P24 +3.3VP, P29 9V S., P32 GND, P33 5V, P34 3,3V, P38 +5VP, P45 GND, P47 9V, U1 DC 9V, U6 LM2940CS-5.0, U7 LM3940IS-3.3

Commit message: megashield_svn_1.3_geschlossen
megashield_svn_1.3_geschlossen
Schönheitsfehler in Plan verbessert
Bei dem globalen Maker "pinRemoteSwitch" war in den Schaltpanseite bei
dem Due die Signalrichtung falsch eingezeichnet.
Signalrichtung wurde  umgeändert
Die Änderung hat kein Einfluß auf die Funktion der Schaltung
Parts:
- C1, C13, C8: symbol CP_Small -> ardumower-mega-shield-svn-rescue:CP_Small-RESCUE-ardumower_mega_shield_svn
- C4, C5, C6, C7: symbol C_Small -> ardumower-mega-shield-svn-rescue:C_Small-RESCUE-ardumower_mega_shield_svn
- D4: symbol D -> ardumower-mega-shield-svn-rescue:D-RESCUE-ardumower_mega_shield_svn
- F1: symbol F_Small -> ardumower-mega-shield-svn-rescue:F_Small-RESCUE-ardumower_mega_shield_svn
- JP1: symbol Jumper_NC_Small -> ardumower-mega-shield-svn-rescue:Jumper_NC_Small-RESCUE-ardumower_mega_shield_svn
- P24, P29, P32, P33, P34, P38, P45, P47: symbol CONN_01X08 -> ardumower-mega-shield-svn-rescue:CONN_01X08-RESCUE-ardumower_mega_shield_svn
- U1: symbol DC-DC_Stepdown -> ardumower-mega-shield-svn-rescue:DC-DC_Stepdown-RESCUE-ardumower_mega_shield_svn
- U6, U7: symbol LM2940CS-5.0 -> ardumower-mega-shield-svn-rescue:LM2940CS-5.0-RESCUE-ardumower_mega_shield_svn
Changed lines of the file:
@@
-EESchema Schematic File Version 2
-LIBS:ardumower mega shield svn-rescue
-LIBS:power
-LIBS:device
-LIBS:Zimprich
-LIBS:conn
-LIBS:transistors
-LIBS:switches
-LIBS:linear
-LIBS:texas
-LIBS:diode
+EESchema Schematic File Version 4
 LIBS:ardumower mega shield svn-cache
 EELAYER 26 0
@@
 $EndDescr
 $Comp
-L DC-DC_Stepdown U1
+L ardumower-mega-shield-svn-rescue:DC-DC_Stepdown-RESCUE-ardumower_mega_shield_svn U1
 U 1 1 57DF681D
 P 2470 1140
@@
 $EndComp
 $Comp
-L CONN_01X08 P33
+L ardumower-mega-shield-svn-rescue:CONN_01X08-RESCUE-ardumower_mega_shield_svn P33
 U 1 1 57DF683D
 P 10135 4410
@@
 $EndComp
 $Comp
-L CONN_01X08 P32
+L ardumower-mega-shield-svn-rescue:CONN_01X08-RESCUE-ardumower_mega_shield_svn P32
 U 1 1 57DF683E
 P 9635 4410
@@
 $EndComp
 $Comp
-L CONN_01X08 P34
+L ardumower-mega-shield-svn-rescue:CONN_01X08-RESCUE-ardumower_mega_shield_svn P34
 U 1 1 57DF683F
 P 10595 4400
@@
 $EndComp
 $Comp
-L GND #PWR0166
+L ardumower-mega-shield-svn-rescue:GND-RESCUE-ardumower_mega_shield_svn #PWR0166
 U 1 1 57DF6841
 P 9435 4810
@@
 Abgriff 5V, 3V, GND
 $Comp
-L CONN_01X08 P47
+L ardumower-mega-shield-svn-rescue:CONN_01X08-RESCUE-ardumower_mega_shield_svn P47
 U 1 1 57DF689F
 P 10605 5490
@@
 Spannungsaufbereitung
 $Comp
-L +9V #PWR0167
+L ardumower-mega-shield-svn-rescue:+9V-RESCUE-ardumower_mega_shield_svn #PWR0167
 U 1 1 57DB0947
 P 10440 5975
@@
 $EndComp
 $Comp
-L +9V #PWR0168
+L ardumower-mega-shield-svn-rescue:+9V-RESCUE-ardumower_mega_shield_svn #PWR0168
 U 1 1 57DB0B58
 P 3620 1575
@@
 $EndComp
 $Comp
-L +5V #PWR0169
+L ardumower-mega-shield-svn-rescue:+5V-RESCUE-ardumower_mega_shield_svn #PWR0169
 U 1 1 57DC5072
 P 10045 4865
@@
 $EndComp
 $Comp
-L +3.3V #PWR0170
+L ardumower-mega-shield-svn-rescue:+3.3V-RESCUE-ardumower_mega_shield_svn #PWR0170
 U 1 1 57DC50AC
 P 10490 4865
@@
 $EndComp
 $Comp
-L GND #PWR0171
+L ardumower-mega-shield-svn-rescue:GND-RESCUE-ardumower_mega_shield_svn #PWR0171
 U 1 1 57DD8587
 P 2820 990
@@
 $EndComp
 $Comp
-L GND #PWR0172
+L ardumower-mega-shield-svn-rescue:GND-RESCUE-ardumower_mega_shield_svn #PWR0172
 U 1 1 57DD8631
 P 2120 990
@@
 $EndComp
 $Comp
-L F_Small F1
+L ardumower-mega-shield-svn-rescue:F_Small-RESCUE-ardumower_mega_shield_svn F1
 U 1 1 57E52B64
 P 3440 1240
@@
 $EndComp
 $Comp
-L D D4
+L ardumower-mega-shield-svn-rescue:D-RESCUE-ardumower_mega_shield_svn D4
 U 1 1 57E52B65
 P 4285 1240
@@
 $EndComp
 $Comp
-L LM2940CS-5.0 U6
+L ardumower-mega-shield-svn-rescue:LM2940CS-5.0-RESCUE-ardumower_mega_shield_svn U6
 U 1 1 57E52B67
 P 6285 1240
@@
 $EndComp
 $Comp
-L CP_Small C1
+L ardumower-mega-shield-svn-rescue:CP_Small-RESCUE-ardumower_mega_shield_svn C1
 U 1 1 57E52B68
 P 4735 1440
@@
 $EndComp
 $Comp
-L C_Small C4
+L ardumower-mega-shield-svn-rescue:C_Small-RESCUE-ardumower_mega_shield_svn C4
 U 1 1 57E52B69
 P 5085 1440
@@
 $EndComp
 $Comp
-L GND #PWR0173
+L ardumower-mega-shield-svn-rescue:GND-RESCUE-ardumower_mega_shield_svn #PWR0173
 U 1 1 57E52B70
 P 7185 2915
@@
 $EndComp
 $Comp
-L CP_Small C8
+L ardumower-mega-shield-svn-rescue:CP_Small-RESCUE-ardumower_mega_shield_svn C8
 U 1 1 57E52B71
 P 7595 1440
@@
 $EndComp
 $Comp
-L C_Small C7
+L ardumower-mega-shield-svn-rescue:C_Small-RESCUE-ardumower_mega_shield_svn C7
 U 1 1 57E52B72
 P 7235 1440
@@
 $EndComp
 $Comp
-L GND #PWR0174
+L ardumower-mega-shield-svn-rescue:GND-RESCUE-ardumower_mega_shield_svn #PWR0174
 U 1 1 57E52B73
 P 7235 1665
@@
 $EndComp
 $Comp
-L LM2940CS-5.0 U7
+L ardumower-mega-shield-svn-rescue:LM2940CS-5.0-RESCUE-ardumower_mega_shield_svn U7
 U 1 1 57E52BA6
 P 6285 2365
@@
 $EndComp
 $Comp
-L C_Small C5
+L ardumower-mega-shield-svn-rescue:C_Small-RESCUE-ardumower_mega_shield_svn C5
 U 1 1 57E52BA7
 P 5185 2515
@@
 $EndComp
 $Comp
-L C_Small C6
+L ardumower-mega-shield-svn-rescue:C_Small-RESCUE-ardumower_mega_shield_svn C6
 U 1 1 57E52BA8
 P 7185 2565
@@
 $EndComp
 $Comp
-L GND #PWR0175
+L ardumower-mega-shield-svn-rescue:GND-RESCUE-ardumower_mega_shield_svn #PWR0175
 U 1 1 57E52BA9
 P 5535 2915
@@
 $EndComp
 $Comp
-L GND #PWR0176
+L ardumower-mega-shield-svn-rescue:GND-RESCUE-ardumower_mega_shield_svn #PWR0176
 U 1 1 57E52BBF
 P 5485 1750
@@
 $EndComp
 $Comp
-L CP_Small C13
+L ardumower-mega-shield-svn-rescue:CP_Small-RESCUE-ardumower_mega_shield_svn C13
 U 1 1 57E52BC0
 P 7605 2565
@@
 $EndComp
 $Comp
-L Jumper_NC_Small JP1
+L ardumower-mega-shield-svn-rescue:Jumper_NC_Small-RESCUE-ardumower_mega_shield_svn JP1
 U 1 1 57E5D727
 P 3100 1240
@@
 Eingang vom 5V Ausgang ?
 $Comp
-L +5VP #PWR0177
+L ardumower-mega-shield-svn-rescue:+5VP-RESCUE-ardumower_mega_shield_svn #PWR0177
 U 1 1 57E9669C
 P 8060 1240
@@
 $EndComp
 $Comp
-L +3.3VP #PWR0178
+L ardumower-mega-shield-svn-rescue:+3.3VP-RESCUE-ardumower_mega_shield_svn #PWR0178
 U 1 1 57E966D4
 P 8065 2365
@@
 $EndComp
 $Comp
-L CONN_01X08 P38
+L ardumower-mega-shield-svn-rescue:CONN_01X08-RESCUE-ardumower_mega_shield_svn P38
 U 1 1 57EFA6BF
 P 9645 1365
@@
 $EndComp
 $Comp
-L CONN_01X08 P24
+L ardumower-mega-shield-svn-rescue:CONN_01X08-RESCUE-ardumower_mega_shield_svn P24
 U 1 1 57EFB361
 P 9095 2685
@@
 $EndComp
 $Comp
-L CONN_01X08 P45
+L ardumower-mega-shield-svn-rescue:CONN_01X08-RESCUE-ardumower_mega_shield_svn P45
 U 1 1 57EFCC69
 P 10155 5485
@@
 $EndComp
 $Comp
-L GND #PWR0179
+L ardumower-mega-shield-svn-rescue:GND-RESCUE-ardumower_mega_shield_svn #PWR0179
 U 1 1 57EFCC6F
 P 9955 5885
@@
 9Vgeschaltet
 $Comp
-L CONN_01X08 P29
+L ardumower-mega-shield-svn-rescue:CONN_01X08-RESCUE-ardumower_mega_shield_svn P29
 U 1 1 58ACC03E
 P 9630 5485
