File: pcb/Produzierte_Platinen/megashield_svn_1.3_geschlossen/USpannungAB.sch (KiCad schematic (older format))
At the start: 15 parts, among them Q2 IRF9540N, Q3 BC817

Commit message: megashield_svn_1.3_geschlossen
megashield_svn_1.3_geschlossen
Schönheitsfehler in Plan verbessert
Bei dem globalen Maker "pinRemoteSwitch" war in den Schaltpanseite bei
dem Due die Signalrichtung falsch eingezeichnet.
Signalrichtung wurde  umgeändert
Die Änderung hat kein Einfluß auf die Funktion der Schaltung
Parts:
- C12: symbol CP1 -> ardumower-mega-shield-svn-rescue:CP1-RESCUE-ardumower_mega_shield_svn
- D12, D13, D14, D15: symbol D -> ardumower-mega-shield-svn-rescue:D-RESCUE-ardumower_mega_shield_svn
- D2: symbol ZENER -> ardumower-mega-shield-svn-rescue:ZENER-RESCUE-ardumower_mega_shield_svn
- JP8: symbol Jumper_NC_Dual -> ardumower-mega-shield-svn-rescue:Jumper_NC_Dual-RESCUE-ardumower_mega_shield_svn
- Q2: symbol IRF9540N-RESCUE-ardumower_mega_shield_svn -> ardumower-mega-shield-svn-rescue:IRF9540N-RESCUE-ardumower_mega_shield_svn
- Q3: symbol BC817-40 -> ardumower-mega-shield-svn-rescue:BC817-40-RESCUE-ardumower_mega_shield_svn
- R32, R33, R34, R35, R36, R37: symbol R -> ardumower-mega-shield-svn-rescue:R-RESCUE-ardumower_mega_shield_svn
Changed lines of the file:
@@
-EESchema Schematic File Version 2
-LIBS:ardumower mega shield svn-rescue
-LIBS:power
-LIBS:device
-LIBS:Zimprich
-LIBS:conn
-LIBS:transistors
-LIBS:switches
-LIBS:linear
-LIBS:texas
-LIBS:diode
+EESchema Schematic File Version 4
 LIBS:ardumower mega shield svn-cache
 EELAYER 26 0
@@
 $EndDescr
 $Comp
-L R R37
+L ardumower-mega-shield-svn-rescue:R-RESCUE-ardumower_mega_shield_svn R37
 U 1 1 57DD94E3
 P 4180 2820
@@
 $EndComp
 $Comp
-L R R32
+L ardumower-mega-shield-svn-rescue:R-RESCUE-ardumower_mega_shield_svn R32
 U 1 1 57DD94E5
 P 5750 3650
@@
 $EndComp
 $Comp
-L R R33
+L ardumower-mega-shield-svn-rescue:R-RESCUE-ardumower_mega_shield_svn R33
 U 1 1 57DD94E7
 P 6255 4155
@@
 $EndComp
 $Comp
-L R R35
+L ardumower-mega-shield-svn-rescue:R-RESCUE-ardumower_mega_shield_svn R35
 U 1 1 57DD94E9
 P 7485 4980
@@
 $EndComp
 $Comp
-L R R34
+L ardumower-mega-shield-svn-rescue:R-RESCUE-ardumower_mega_shield_svn R34
 U 1 1 57DD94EA
 P 6255 4795
@@
 $EndComp
 $Comp
-L CP1 C12
+L ardumower-mega-shield-svn-rescue:CP1-RESCUE-ardumower_mega_shield_svn C12
 U 1 1 57DD94EC
 P 6255 5440
@@
 $EndComp
 $Comp
-L GND #PWR0216
+L ardumower-mega-shield-svn-rescue:GND-RESCUE-ardumower_mega_shield_svn #PWR0216
 U 1 1 57DD94ED
 P 7030 6010
@@
 vielleicht schreibst du noch bei was die teilschaltungen machen sollen\n[00:05:52] Alexander Grau: zener diode z.b. soll Ugs auf -15 volt begrenzen\n[00:06:31] Alexander Grau: C9 und D13 sollen über R31, R30 eine verzögerungsschaltung bilden\n[00:06:39] Alexander Grau: (für eine richtung)\n[00:07:27] Alexander Grau: beim pmos evtl. noch beschreiben wann er schaltet und wann nicht:\n[00:07:37] Alexander Grau: Ugs=-15v (pmos schaltet)\n[00:07:43] Alexander Grau: Ugs=0v (pmos schaltet nicht)\n[00:08:14] Alexander Grau: dann versteht man die schaltung besser :)\n[00:08:22] Kurzschuss - Uwe -: die Zeit reicht auf alle fälle oder sollte da evl noch ein Poti vorgesehen werden\n[00:08:37] Alexander Grau: 3 sek reichen dicke - eigentlich reicht schon 1 sek
 $Comp
-L R R36
+L ardumower-mega-shield-svn-rescue:R-RESCUE-ardumower_mega_shield_svn R36
 U 1 1 57DD94F0
 P 8025 4195
@@
 beim flashen über usb wird der akku getrennt (alle pins gehen auf hochomig) - das sollte aber kein problem sein (usb versorgung des arduinos) - beim programmstart wird der akku dann wieder zugeschaltet
 $Comp
-L ZENER D2
+L ardumower-mega-shield-svn-rescue:ZENER-RESCUE-ardumower_mega_shield_svn D2
 U 1 1 57DDA0D5
 P 4555 2870
@@
 $EndComp
 $Comp
-L D D14
+L ardumower-mega-shield-svn-rescue:D-RESCUE-ardumower_mega_shield_svn D14
 U 1 1 57DDCD22
 P 6630 1945
@@
 Connection ~ 3090 2470
 $Comp
-L D D13
+L ardumower-mega-shield-svn-rescue:D-RESCUE-ardumower_mega_shield_svn D13
 U 1 1 57E85F65
 P 6255 3020
@@
 $EndComp
 $Comp
-L D D15
+L ardumower-mega-shield-svn-rescue:D-RESCUE-ardumower_mega_shield_svn D15
 U 1 1 57E86A66
 P 6650 3650
@@
 $EndComp
 $Comp
-L D D12
+L ardumower-mega-shield-svn-rescue:D-RESCUE-ardumower_mega_shield_svn D12
 U 1 1 57E89203
 P 5905 4790
@@
 $EndComp
 $Comp
-L BC817-40 Q3
+L ardumower-mega-shield-svn-rescue:BC817-40-RESCUE-ardumower_mega_shield_svn Q3
 U 1 1 57E98AAA
 P 7130 4195
@@
 $EndComp
 $Comp
-L IRF9540N-RESCUE-ardumower_mega_shield_svn Q2
+L ardumower-mega-shield-svn-rescue:IRF9540N-RESCUE-ardumower_mega_shield_svn Q2
 U 1 1 57E9B1CB
 P 3780 3700
@@
 $EndComp
 $Comp
-L Jumper_NC_Dual JP8
+L ardumower-mega-shield-svn-rescue:Jumper_NC_Dual-RESCUE-ardumower_mega_shield_svn JP8
 U 1 1 5834DE11
 P 8430 4195
