File: pcb/Produzierte_Platinen/megashield_svn_1.3_geschlossen/VerpolungsschutzLade.sch (KiCad schematic (older format))
At the start: 3 parts, among them Q4 IRF9540N

Commit message: megashield_svn_1.3_geschlossen
megashield_svn_1.3_geschlossen
Schönheitsfehler in Plan verbessert
Bei dem globalen Maker "pinRemoteSwitch" war in den Schaltpanseite bei
dem Due die Signalrichtung falsch eingezeichnet.
Signalrichtung wurde  umgeändert
Die Änderung hat kein Einfluß auf die Funktion der Schaltung
Parts:
- D7: symbol ZENER -> ardumower-mega-shield-svn-rescue:ZENER-RESCUE-ardumower_mega_shield_svn
- Q4: symbol IRF9540N-RESCUE-ardumower_mega_shield_svn -> ardumower-mega-shield-svn-rescue:IRF9540N-RESCUE-ardumower_mega_shield_svn
- R57: symbol R_Small -> ardumower-mega-shield-svn-rescue:R_Small-RESCUE-ardumower_mega_shield_svn
Changed lines of the file:
@@
-EESchema Schematic File Version 2
-LIBS:ardumower mega shield svn-rescue
-LIBS:power
-LIBS:device
-LIBS:Zimprich
-LIBS:conn
-LIBS:transistors
-LIBS:switches
-LIBS:linear
-LIBS:texas
-LIBS:diode
+EESchema Schematic File Version 4
 LIBS:ardumower mega shield svn-cache
 EELAYER 26 0
@@
 $EndDescr
 $Comp
-L R_Small R57
+L ardumower-mega-shield-svn-rescue:R_Small-RESCUE-ardumower_mega_shield_svn R57
 U 1 1 57E64A6C
 P 4905 3410
@@
 $EndComp
 $Comp
-L ZENER D7
+L ardumower-mega-shield-svn-rescue:ZENER-RESCUE-ardumower_mega_shield_svn D7
 U 1 1 57E64BD0
 P 5290 3010
@@
 	4480 2755 4655 2755
 $Comp
-L GND #PWR0273
+L ardumower-mega-shield-svn-rescue:GND-RESCUE-ardumower_mega_shield_svn #PWR0273
 U 1 1 57E64EC6
 P 4905 3620
@@
 d7 geändert\nvon ZPD15 auf\nSMD ZF 15
 $Comp
-L IRF9540N-RESCUE-ardumower_mega_shield_svn Q4
+L ardumower-mega-shield-svn-rescue:IRF9540N-RESCUE-ardumower_mega_shield_svn Q4
 U 1 1 57E9A340
 P 4855 2855
