Commit message: introduced ardumower ros package

File: code/ros/ardumower/robot/robot.urdf (robot description, URDF)
Before this commit: robot test_robot, 6 links, 5 joints
Links:
- added link imu_link; visual box size=.03 .015 .01
- link base_link: geometry visual box size=0.5 0.32 0.25
- link fwheel_attach: geometry visual cylinder length=0.060 radius=0.1
- link lwheel: geometry visual cylinder length=0.008 radius=0.13
- link rwheel: geometry visual cylinder length=0.008 radius=0.13
- link scanner: geometry visual box size=0.1 0.1 0.015
Joints:
- added joint base_to_imu: type fixed, parent base_link, child imu_link, origin xyz=0.105 0 0.17 rpy=0 0 0
- joint base_to_fwheel: origin xyz=0.13 0 0.02 rpy=0 0 0 -> xyz=0.5 0 0.02 rpy=0 0 0
- joint base_to_lwheel: origin xyz=0 0.115 0.046 rpy=1.5708 0 0 -> xyz=0 0.22 0.13 rpy=1.5708 0 0
- joint base_to_rwheel: origin xyz=0 -0.115 0.046 rpy=-1.5708 0 0 -> xyz=0 -0.22 0.13 rpy=-1.5708 0 0
- joint base_to_scanner: origin xyz=0.105 0 0.22 rpy=0 0 0 -> xyz=0.26 0 0.46 rpy=0 0 1.57
