File: pcb/Test_und_Entwicklung/megashield_svn_1.4_geoeffnet/Spannungsversorgung.kicad_sch (KiCad schematic)
At the start: 21 parts, among them P24 +3.3VP, P29 9V S., P32 GND, P33 5V, P34 3,3V, P38 +5VP, P45 GND, P47 9V, U1 DC 9V, U6 LM2940CS-5.0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

Commit message: megashield_svn_1.4_geoeffnet
megashield_svn_1.4_geoeffnet
5 EF3 Footprint geaendert
Parts:
- F1: footprint SMD_Packages:Fuse_SMD -> Zimprich:Fuse_SMD
Changed lines of the file:
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@@
       (effects (font (size 1.27 1.27)) (justify left))
     )
-    (property "Footprint" "SMD_Packages:Fuse_SMD" (id 2) (at 87.376 31.496 0)
+    (property "Footprint" "Zimprich:Fuse_SMD" (id 2) (at 87.376 31.496 0)
       (effects (font (size 1.524 1.524)) hide)
     )

Commit message: megashield_svn_1.4_geoeffnet
megashield_svn_1.4_geoeffnet
11 Sicherheitskopie alles fertig gezeichnet
Parts:
- C4, C5, C6, C7: Bestelllink (none) -> https://www.reichelt.de/de/en/mlcc-0805-100nf-100v-10-ft-ca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; Bestücken (Assemble) (none) -> JA (YES); Funktion (none) -> X7R 0805FCG 100N MLCC, 0805, 100nF, 100V, 10%, FT-Cap
- D4: Bestücken (Assemble) (none) -> JA (YES); Funktion Value -> Gleichrichterdiode, 400 V, 1 A, DO-214AC/SMA; Reichelt-Bestellnummer (none) -> R: S 1G SMD
- F1: Bestellnummer Value -> R: OMH 125 HALTER; Bestücken (Assemble) (none) -> JA (YES)
- U6: Bestelllink (none) -> https://www.reichelt.de/de/en/ldo-voltage-regulator-5v-to-2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; Bestellnummer (none) -> R: LM 2940 CS-5.0; Bestücken (Assemble) (none) -> JA (YES); Funktion (none) -> LDO voltage regulator 5V TO-263-3; Gehäuseart (none) -> TO-263-3; Reichelt-Bestellnummer (none) -> R: LM 2940 CS-5.0; Technische Daten (none) -> LDO voltage regulator 5V TO-263-3
- U7: Bestelllink Value -> https://www.reichelt.de/de/en/ldo-voltage-regulator-fixed-3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; Bestellnummer Value -> R: LM 3940 IS3,3; Bestücken (Assemble) (none) -> JA (YES); Funktion (none) -> LDO voltage regulator, fixed, 3.3 Vout, 1 A, D2PAK; Gehäuseart Value -> D²PAK; Reichelt-Bestellnummer (none) -> R: LM 3940 IS3,3; Technische Daten Value -> LDO voltage regulator, fixed, 3.3 Vout, 1 A, D2PAK
Changed lines of the file:
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@@
 (kicad_sch (version 20201015) (generator eeschema)
-  (page 1 34)
   (paper "A4")
   (title_block
@@
       (effects (font (size 1.524 1.524)) hide)
     )
-    (property "Bestellnummer" "Value" (id 7) (at 87.376 31.496 0)
+    (property "Bestellnummer" "R: OMH 125 HALTER" (id 7) (at 87.376 31.496 0)
       (effects (font (size 1.524 1.524)) hide)
     )
@@
     (property "Hersteller Bestellnummer" "Value" (id 11) (at 87.376 31.496 0)
       (effects (font (size 1.524 1.524)) hide)
+    )
+    (property "Bestücken (Assemble)" "JA (YES)" (id 4) (at 87.376 31.496 0)
+      (effects (font (size 1.27 1.27)) hide)
     )
   )
@@
       (effects (font (size 1.524 1.524)))
     )
+    (property "Bestelllink" "https://www.reichelt.de/de/en/mlcc-0805-100nf-100v-10-ft-cap-x7r-0805fcg-100n-p193842.html?GROUPID=8048&SEARCH=0805%2B100nf&&r=1" (id 4) (at 129.159 36.576 0)
+      (effects (font (size 1.27 1.27)) hide)
+    )
+    (property "Bestücken (Assemble)" "JA (YES)" (id 5) (at 129.159 36.576 0)
+      (effects (font (size 1.27 1.27)) hide)
+    )
+    (property "Funktion" "X7R 0805FCG 100N MLCC, 0805, 100nF, 100V, 10%, FT-Cap" (id 6) (at 129.159 36.576 0)
+      (effects (font (size 1.27 1.27)) hide)
+    )
   )
   (symbol (lib_id "ardumower-mega-shield-svn-rescue:C_Small-RESCUE-ardumower_mega_shield_svn") (at 131.699 63.881 0) (unit 1)
@@
       (effects (font (size 1.524 1.524)))
     )
+    (property "Bestelllink" "https://www.reichelt.de/de/en/mlcc-0805-100nf-100v-10-ft-cap-x7r-0805fcg-100n-p193842.html?GROUPID=8048&SEARCH=0805%2B100nf&&r=1" (id 4) (at 131.699 63.881 0)
+      (effects (font (size 1.27 1.27)) hide)
+    )
+    (property "Bestücken (Assemble)" "JA (YES)" (id 5) (at 131.699 63.881 0)
+      (effects (font (size 1.27 1.27)) hide)
+    )
+    (property "Funktion" "X7R 0805FCG 100N MLCC, 0805, 100nF, 100V, 10%, FT-Cap" (id 6) (at 131.699 63.881 0)
+      (effects (font (size 1.27 1.27)) hide)
+    )
   )
   (symbol (lib_id "ardumower-mega-shield-svn-rescue:C_Small-RESCUE-ardumower_mega_shield_svn") (at 182.499 65.151 0) (unit 1)
@@
       (effects (font (size 1.524 1.524)))
     )
+    (property "Bestelllink" "https://www.reichelt.de/de/en/mlcc-0805-100nf-100v-10-ft-cap-x7r-0805fcg-100n-p193842.html?GROUPID=8048&SEARCH=0805%2B100nf&&r=1" (id 4) (at 182.499 65.151 0)
+      (effects (font (size 1.27 1.27)) hide)
+    )
+    (property "Bestücken (Assemble)" "JA (YES)" (id 5) (at 182.499 65.151 0)
+      (effects (font (size 1.27 1.27)) hide)
+    )
+    (property "Funktion" "X7R 0805FCG 100N MLCC, 0805, 100nF, 100V, 10%, FT-Cap" (id 6) (at 182.499 65.151 0)
+      (effects (font (size 1.27 1.27)) hide)
+    )
   )
   (symbol (lib_id "ardumower-mega-shield-svn-rescue:C_Small-RESCUE-ardumower_mega_shield_svn") (at 183.769 36.576 0) (unit 1)
@@
     (property "Datasheet" "" (id 3) (at 183.769 36.576 0)
       (effects (font (size 1.524 1.524)))
+    )
+    (property "Bestelllink" "https://www.reichelt.de/de/en/mlcc-0805-100nf-100v-10-ft-cap-x7r-0805fcg-100n-p193842.html?GROUPID=8048&SEARCH=0805%2B100nf&&r=1" (id 4) (at 183.769 36.576 0)
+      (effects (font (size 1.27 1.27)) hide)
+    )
+    (property "Bestücken (Assemble)" "JA (YES)" (id 5) (at 183.769 36.576 0)
+      (effects (font (size 1.27 1.27)) hide)
+    )
+    (property "Funktion" "X7R 0805FCG 100N MLCC, 0805, 100nF, 100V, 10%, FT-Cap" (id 6) (at 183.769 36.576 0)
+      (effects (font (size 1.27 1.27)) hide)
     )
   )
@@
       (effects (font (size 1.524 1.524)) hide)
     )
-    (property "Funktion" "Value" (id 9) (at 108.839 31.496 0)
+    (property "Funktion" "Gleichrichterdiode, 400 V, 1 A, DO-214AC/SMA" (id 9) (at 108.839 31.496 0)
       (effects (font (size 1.524 1.524)) hide)
     )
@@
     (property "Hersteller Bestellnummer" "Value" (id 11) (at 108.839 31.496 0)
       (effects (font (size 1.524 1.524)) hide)
+    )
+    (property "Bestücken (Assemble)" "JA (YES)" (id 4) (at 108.839 31.496 0)
+      (effects (font (size 1.27 1.27)) hide)
+    )
+    (property "Reichelt-Bestellnummer" "R: S 1G SMD" (id 4) (at 108.839 31.496 0)
+      (effects (font (size 1.27 1.27)) hide)
     )
   )
@@
       (effects (font (size 1.524 1.524)))
     )
+    (property "Bestelllink" "https://www.reichelt.de/de/en/ldo-voltage-regulator-5v-to-263-3-lm-2940-cs-5-0-p187697.html?GROUPID=5466&SEARCH=LM2940CS-5.0&&r=1" (id 4) (at 159.639 31.496 0)
+      (effects (font (size 1.27 1.27)) hide)
+    )
+    (property "Bestellnummer" "R: LM 2940 CS-5.0" (id 5) (at 159.639 31.496 0)
+      (effects (font (size 1.27 1.27)) hide)
+    )
+    (property "Bestücken (Assemble)" "JA (YES)" (id 6) (at 159.639 31.496 0)
+      (effects (font (size 1.27 1.27)) hide)
+    )
+    (property "Funktion" "LDO voltage regulator 5V TO-263-3" (id 7) (at 159.639 31.496 0)
+      (effects (font (size 1.27 1.27)) hide)
+    )
+    (property "Gehäuseart" "TO-263-3 " (id 8) (at 159.639 31.496 0)
+      (effects (font (size 1.27 1.27)) hide)
+    )
+    (property "Reichelt-Bestellnummer" "R: LM 2940 CS-5.0" (id 9) (at 159.639 31.496 0)
+      (effects (font (size 1.27 1.27)) hide)
+    )
+    (property "Technische Daten" "LDO voltage regulator 5V TO-263-3" (id 10) (at 159.639 31.496 0)
+      (effects (font (size 1.27 1.27)) hide)
+    )
   )
   (symbol (lib_id "ardumower-mega-shield-svn-rescue:LM2940CS-5.0-RESCUE-ardumower_mega_shield_svn") (at 159.639 60.071 0) (unit 1)
@@
       (effects (font (size 1.524 1.524)) hide)
     )
-    (property "Gehäuseart" "Value" (id 4) (at 159.639 60.071 0)
-      (effects (font (size 1.524 1.524)) hide)
-    )
-    (property "Bestelllink" "Value" (id 5) (at 159.639 60.071 0)
-      (effects (font (size 1.524 1.524)) hide)
-    )
-    (property "Technische Daten" "Value" (id 6) (at 159.639 60.071 0)
-      (effects (font (size 1.524 1.524)) hide)
-    )
-    (property "Bestellnummer" "Value" (id 7) (at 159.639 60.071 0)
+    (property "Gehäuseart" "D²PAK " (id 4) (at 159.639 60.071 0)
+      (effects (font (size 1.524 1.524)) hide)
+    )
+    (property "Bestelllink" "https://www.reichelt.de/de/en/ldo-voltage-regulator-fixed-3-3-vout-1-a-d2pak-lm-3940-is3-3-p109408.html?GROUPID=5466&SEARCH=LM3940IS-3.3&&r=1" (id 5) (at 159.639 60.071 0)
+      (effects (font (size 1.524 1.524)) hide)
+    )
+    (property "Technische Daten" "LDO voltage regulator, fixed, 3.3 Vout, 1 A, D2PAK" (id 6) (at 159.639 60.071 0)
+      (effects (font (size 1.524 1.524)) hide)
+    )
+    (property "Bestellnummer" "R: LM 3940 IS3,3" (id 7) (at 159.639 60.071 0)
       (effects (font (size 1.524 1.524)) hide)
     )
@@
       (effects (font (size 1.524 1.524)) hide)
     )
-  )
+    (property "Bestücken (Assemble)" "JA (YES)" (id 4) (at 159.639 60.071 0)
+      (effects (font (size 1.27 1.27)) hide)
+    )
+    (property "Funktion" "LDO voltage regulator, fixed, 3.3 Vout, 1 A, D2PAK" (id 5) (at 159.639 60.071 0)
+      (effects (font (size 1.27 1.27)) hide)
+    )
+    (property "Reichelt-Bestellnummer" "R: LM 3940 IS3,3" (id 6) (at 159.639 60.071 0)
+      (effects (font (size 1.27 1.27)) hide)
+    )
+  )

Commit message: megashield_svn_1.4_geoeffnet
megashield_svn_1.4_geoeffnet
12 Bauteile Links hinzugefügt
Parts:
- C1, C13, C8: value 22uF -> 22uF / 63V; Bauform Value -> 6,3x11mm, RM 2,5mm; Bestelllink Value -> https://www.reichelt.de/de/en/electrolytic-capacitor-6-3-x-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; Bestellnummer Value -> R: RAD 22/63; Bestücken (Assemble) (none) -> NEIN (NO); Funktion Value -> Elko, radial, 22 µF, 63 V, RM 2,5, 85°C, 2000h, 20%; Hersteller Value -> (none); Hersteller Bestellnummer Value -> (none); Reichelt-Bestellnummer (none) -> R: RAD 22/63; Technische Daten Value -> Elko, radial, 22 µF, 63 V, RM 2,5, 85°C, 2000h, 20%
- C4, C5, C6, C7: Bestellnummer (none) -> Value; Gehäuseart (none) -> Value
- JP1, P24, P29, P32, P33, P34, P38, P45, P47: Bestücken (Assemble) (none) -> NEIN (NO)
- U1: Bestücken (Assemble) (none) -> NEIN (NO); Gehäuseart Value -> (none)

Commit message: megashield_svn_1.4_geoeffnet
megashield_svn_1.4_geoeffnet
19 Feinsicherungshalter mit SMD Sicherungshalter ausgetauscht
Parts:
- F1: Funktion Value -> OMH 125 HALTER SMD-Sicherungshalter für OMT-125; Reichelt-Bestellnummer (none) -> R: OMH 125 HALTER; Technische Daten https://www.reichelt.de/SMD-Sicherungen/OMH-125-HALTER/3/in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 -> OMH 125 HALTER SMD-Sicherungshalter für OMT-125
Changed lines of the file:
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@@
       (effects (font (size 1.524 1.524)) hide)
     )
-    (property "Technische Daten" "https://www.reichelt.de/SMD-Sicherungen/OMH-125-HALTER/3/index.html?ACTION=3&LA=446&ARTICLE=77866&GROUPID=7660&artnr=OMH+125+HALTER&SEARCH=smd%2Bsicherung%2B125" (id 6) (at 87.376 31.496 0)
+    (property "Technische Daten" "OMH 125 HALTER SMD-Sicherungshalter für OMT-125" (id 6) (at 87.376 31.496 0)
       (effects (font (size 1.524 1.524)) hide)
     )
@@
       (effects (font (size 1.524 1.524)) hide)
     )
-    (property "Funktion" "Value" (id 9) (at 87.376 31.496 0)
+    (property "Funktion" "OMH 125 HALTER SMD-Sicherungshalter für OMT-125" (id 9) (at 87.376 31.496 0)
       (effects (font (size 1.524 1.524)) hide)
     )
@@
       (effects (font (size 1.27 1.27)) hide)
     )
+    (property "Reichelt-Bestellnummer" "R: OMH 125 HALTER" (id 4) (at 87.376 31.496 0)
+      (effects (font (size 1.27 1.27)) hide)
+    )
