File: pcb/Test_und_Entwicklung/megashield_svn_1.4_geoeffnet/LShifter3.kicad_sch (KiCad schematic)
At the start: 3 parts, among them Q7 BSS138

Commit message: megashield_svn_1.4_geoeffnet
megashield_svn_1.4_geoeffnet
24 INA Neu verdrahtet und Widerstandswerte von den INA ausgetauscht
Berechnung hinzugefügt
Parts:
- Q7: JLCPCB LCSC Part (none) -> C426569
- R62, R63: Bestücken (Assemble) JA (YES) -> (none); JLCPCB LCSC Part (none) -> C25804

Commit message: megashield_svn_1.4_geoeffnet
megashield_svn_1.4_geoeffnet
28 Beschriftung von Deutsch auf Englisch umgeändert
Parts:
- Q7: Bauform Value -> (none); JLCPCB LCSC Part C426569 -> (none)
- R62, R63: Bauform Value -> (none); Bestücken (Assemble) (none) -> JA (YES); JLCPCB LCSC Part C25804 -> (none)

Commit message: megashield_svn_1.4_geoeffnet
megashield_svn_1.4_geoeffnet
29 BY1-BY12 JLCCPCB Nummer ergänzt
Parts:
- Q7: JLCPCB Basic / Extern (none) -> 1; JLCPCB LCSC Part (none) -> C426569
- R62, R63: JLCPCB LCSC Part (none) -> C17902
Changed lines of the file:
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@@
       (effects (font (size 1.524 1.524)) (justify left) hide)
     )
-    (property "JLCPCB LCSC Part" "" (id 9) (at 138.049 82.55 0)
+    (property "JLCPCB LCSC Part" "C17902" (id 9) (at 138.049 82.55 0)
       (effects (font (size 1.27 1.27)) hide)
     )
@@
       (effects (font (size 1.524 1.524)) (justify left) hide)
     )
-    (property "JLCPCB LCSC Part" "" (id 9) (at 155.194 82.55 0)
+    (property "JLCPCB LCSC Part" "C17902" (id 9) (at 155.194 82.55 0)
       (effects (font (size 1.27 1.27)) hide)
     )
@@
       (effects (font (size 1.27 1.27)) hide)
     )
-    (property "JLCPCB LCSC Part" "" (id 7) (at 147.447 92.329 0)
+    (property "JLCPCB LCSC Part" "C426569" (id 7) (at 147.447 92.329 0)
       (effects (font (size 1.27 1.27)) hide)
     )
+    (property "JLCPCB Basic / Extern" "1" (id 8) (at 147.447 92.329 0)
+      (effects (font (size 1.27 1.27)) hide)
+    )
