File: pcb/Test_und_Entwicklung/megashield_svn_1.4_geoeffnet/LShifter9.kicad_sch (KiCad schematic)
At the start: 3 parts, among them Q31 BSS138

Commit message: megashield_svn_1.4_geoeffnet
megashield_svn_1.4_geoeffnet
24 INA Neu verdrahtet und Widerstandswerte von den INA ausgetauscht
Berechnung hinzugefügt
Parts:
- Q31: JLCPCB LCSC Part (none) -> C426569
- R100, R99: Bestücken (Assemble) JA (YES) -> (none); JLCPCB LCSC Part (none) -> C25804

Commit message: megashield_svn_1.4_geoeffnet
megashield_svn_1.4_geoeffnet
28 Beschriftung von Deutsch auf Englisch umgeändert
Parts:
- Q31: Bauform Value -> (none); JLCPCB LCSC Part C426569 -> (none)
- R100, R99: Bauform Value -> (none); Bestücken (Assemble) (none) -> JA (YES); JLCPCB LCSC Part C25804 -> (none)

Commit message: megashield_svn_1.4_geoeffnet
megashield_svn_1.4_geoeffnet
29 BY1-BY12 JLCCPCB Nummer ergänzt
Parts:
- Q31: JLCPCB Basic / Extern (none) -> 1; JLCPCB LCSC Part (none) -> C426569
- R100, R99: JLCPCB LCSC Part (none) -> C17902
