File: pcb/Test_und_Entwicklung/megashield_svn_1.4_geoeffnet/LShifter7.kicad_sch (KiCad schematic)
At the start: 3 parts, among them Q11 BSS138

Commit message: megashield_svn_1.4_geoeffnet
megashield_svn_1.4_geoeffnet
33 Q5-Q11,Q30-Q37 neue JLCPCB Nummer und neue Herstellernummer BSS138 (2n7002)
Parts:
- Q11: value BSS138 -> BSS138 (2n7002); JLCPCB Basic / Extern 1 -> (none); JLCPCB LCSC Part C426569 -> C8545

Commit message: megashield_svn_1.4_geoeffnet
megashield_svn_1.4_geoeffnet
41 Q24 + R6 hinzugefügt und Summer ansteuerung umgeändert
Other:
- company: ML AG JL UZ -> ML AG JL BS UZ
