File: pcb/Test_und_Entwicklung/megashield_svn_1.4_geoeffnet/MotorRechts.kicad_sch (KiCad schematic)
At the start: 6 parts

Commit message: megashield_svn_1.4_geoeffnet
megashield_svn_1.4_geoeffnet
29 BY1-BY12 JLCCPCB Nummer ergänzt
Parts:
- BY10, BY11, BY12, BY9: JLCPCB Basic / Extern (none) -> 1; JLCPCB LCSC Part (none) -> C123929
- CC3: Bestücken (Assemble) JA (YES) -> (none); Funktion Film Capacitors 250V .01uF 5% TOL MAX REFLOW 250/C -> (none); JLCPCB Basic / Extern (none) -> 1; JLCPCB LCSC Part (none) -> C53737
- RL3: JLCPCB Basic / Extern (none) -> 1; JLCPCB LCSC Part (none) -> C25473
Changed lines of the file:
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@@
       (effects (font (size 1.27 1.27)) hide)
     )
-    (property "Gehäuseart" "2512" (id 4) (at 110.49 98.298 0)
+    (property "Gehäuseart" "2512" (id 5) (at 110.49 98.298 0)
+      (effects (font (size 1.27 1.27)) hide)
+    )
+    (property "JLCPCB Basic / Extern" "1" (id 6) (at 110.49 98.298 0)
+      (effects (font (size 1.27 1.27)) hide)
+    )
+    (property "JLCPCB LCSC Part" "C25473" (id 7) (at 110.49 98.298 0)
       (effects (font (size 1.27 1.27)) hide)
     )
@@
       (effects (font (size 1.524 1.524)) hide)
     )
-    (property "JLCPCB LCSC Part" "" (id 9) (at 80.518 90.805 0)
+    (property "JLCPCB LCSC Part" "C123929" (id 9) (at 80.518 90.805 0)
       (effects (font (size 1.27 1.27)) hide)
     )
@@
       (effects (font (size 1.27 1.27)) hide)
     )
+    (property "JLCPCB Basic / Extern" "1" (id 9) (at 80.518 90.805 0)
+      (effects (font (size 1.27 1.27)) hide)
+    )
   )
   (symbol (lib_id "ardumower-mega-shield-svn-rescue:D-RESCUE-ardumower_mega_shield_svn") (at 80.518 104.902 90) (mirror x) (unit 1)
@@
       (effects (font (size 1.524 1.524)) hide)
     )
-    (property "JLCPCB LCSC Part" "" (id 9) (at 80.518 104.902 0)
+    (property "JLCPCB LCSC Part" "C123929" (id 9) (at 80.518 104.902 0)
       (effects (font (size 1.27 1.27)) hide)
     )
@@
       (effects (font (size 1.27 1.27)) hide)
     )
+    (property "JLCPCB Basic / Extern" "1" (id 9) (at 80.518 104.902 0)
+      (effects (font (size 1.27 1.27)) hide)
+    )
   )
   (symbol (lib_id "ardumower-mega-shield-svn-rescue:D-RESCUE-ardumower_mega_shield_svn") (at 124.333 90.805 270) (unit 1)
@@
       (effects (font (size 1.524 1.524)) hide)
     )
-    (property "JLCPCB LCSC Part" "" (id 9) (at 124.333 90.805 0)
+    (property "JLCPCB LCSC Part" "C123929" (id 9) (at 124.333 90.805 0)
       (effects (font (size 1.27 1.27)) hide)
     )
@@
       (effects (font (size 1.27 1.27)) hide)
     )
+    (property "JLCPCB Basic / Extern" "1" (id 9) (at 124.333 90.805 0)
+      (effects (font (size 1.27 1.27)) hide)
+    )
   )
   (symbol (lib_id "ardumower-mega-shield-svn-rescue:D-RESCUE-ardumower_mega_shield_svn") (at 124.333 105.029 270) (unit 1)
@@
       (effects (font (size 1.524 1.524)) hide)
     )
-    (property "JLCPCB LCSC Part" "" (id 9) (at 124.333 105.029 0)
+    (property "JLCPCB LCSC Part" "C123929" (id 9) (at 124.333 105.029 0)
       (effects (font (size 1.27 1.27)) hide)
     )
@@
     )
     (property "Bestücken (Assemble)" "JA (YES)" (id 8) (at 124.333 105.029 0)
+      (effects (font (size 1.27 1.27)) hide)
+    )
+    (property "JLCPCB Basic / Extern" "1" (id 9) (at 124.333 105.029 0)
       (effects (font (size 1.27 1.27)) hide)
     )
@@
       (effects (font (size 1.27 1.27)) hide)
     )
-    (property "Bestücken (Assemble)" "JA (YES)" (id 4) (at 91.948 98.298 0)
-      (effects (font (size 1.27 1.27)) hide)
-    )
-    (property "Funktion" "Film Capacitors 250V .01uF 5% TOL MAX REFLOW 250/C" (id 5) (at 91.948 98.298 0)
-      (effects (font (size 1.27 1.27)) hide)
-    )
-    (property "Bauform" "" (id 6) (at 91.948 98.298 0)
-      (effects (font (size 1.27 1.27)) hide)
-    )
-    (property "Bestellnummer" "Value" (id 7) (at 91.948 98.298 0)
-      (effects (font (size 1.27 1.27)) hide)
-    )
+    (property "JLCPCB Basic / Extern" "1" (id 8) (at 91.948 98.298 0)
+      (effects (font (size 1.27 1.27)) hide)
+    )
+    (property "JLCPCB LCSC Part" "C53737" (id 9) (at 91.948 98.298 0)
+      (effects (font (size 1.27 1.27)) hide)
+    )
+    (property "Bauform" "" (id 4) (at 91.948 98.298 0)
+      (effects (font (size 1.27 1.27)) hide)
+    )
+    (property "Bestellnummer" "Value" (id 5) (at 91.948 98.298 0)
+      (effects (font (size 1.27 1.27)) hide)
+    )

Commit message: megashield_svn_1.4_geoeffnet
megashield_svn_1.4_geoeffnet
38 D3 Bauform geändert auf 0805 + neue JLCPCB Nummer
Parts:
- CC3: Bestücken (Assemble) (none) -> JA (YES)
Changed lines of the file:
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@@
+      (effects (font (size 1.27 1.27)) hide)
+    )
+    (property "Bestücken (Assemble)" "JA (YES)" (id 6) (at 91.948 98.298 0)
       (effects (font (size 1.27 1.27)) hide)
     )

Commit message: megashield_svn_1.4_geoeffnet
megashield_svn_1.4_geoeffnet
39 CC1,CC2,CC3 Footprint auf 1206 geändert
Parts:
- CC3: footprint Capacitor_SMD:C_2220_5650Metric -> Capacitor_SMD:C_1206_3216Metric; Gehäuseart 2220 -> 1206
Changed lines of the file:
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@@
     (property "Reference" "CC3" (id 0) (at 91.948 91.8972 90))
     (property "Value" "SMDIF02100QA00JQ00 " (id 1) (at 91.948 94.2086 90))
-    (property "Footprint" "Capacitor_SMD:C_2220_5650Metric" (id 2) (at 89.0524 95.377 0)
+    (property "Footprint" "Capacitor_SMD:C_1206_3216Metric" (id 2) (at 89.0524 95.377 0)
       (effects (font (size 1.27 1.27)) (justify left) hide)
     )
@@
       (effects (font (size 1.27 1.27)) (justify left) hide)
     )
-    (property "Gehäuseart" "2220" (id 4) (at 91.567 95.377 0)
+    (property "Gehäuseart" "1206" (id 4) (at 91.567 95.377 0)
       (effects (font (size 1.524 1.524)) (justify left) hide)
     )

Commit message: megashield_svn_1.4_geoeffnet
megashield_svn_1.4_geoeffnet
41 Q24 + R6 hinzugefügt und Summer ansteuerung umgeändert
Other:
- company: ML AG JL UZ -> ML AG JL BS UZ
Changed lines of the file:
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@@
   (title_block
     (title "Ardumower shield SVN Version")
-    (date "2021-01-07")
+    (date "2021-01-11")
     (rev "1.4")
-    (company "ML AG JL UZ")
-    (comment 1 "Unterspannungsschutz von AlexanderG")
+    (company "ML AG JL BS UZ")
+    (comment 1 "Schaltplan und Layout UweZ")
   )
   (junction (at 80.518 98.298) (diameter 0.9144) (color 0 0 0 0))

Commit message: megashield_svn_1.4_geoeffnet
megashield_svn_1.4_geoeffnet
43 neue JLCPCB Nummer Für CC1,CC2,CC3,EF1,U4,U9,U12,U6,U7,PC1-PC7
Parts:
- CC3: JLCPCB LCSC Part C53737 -> C1944
Changed lines of the file:
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@@
       (effects (font (size 1.27 1.27)) hide)
     )
-    (property "JLCPCB LCSC Part" "C53737" (id 9) (at 91.948 98.298 0)
+    (property "JLCPCB LCSC Part" "C1944" (id 9) (at 91.948 98.298 0)
       (effects (font (size 1.27 1.27)) hide)
     )
