File: pcb/Test_und_Entwicklung/megashield_svn_1.4_Prototyp_Intern_geschlossen/LShifter14.kicad_sch (KiCad schematic)
At the start: 3 parts, among them Q36 BSS138 (2n7002)

Commit message: megashield_svn_1.4_Prototyp_Intern_geschlossen
megashield_svn_1.4_Prototyp_Intern_geschlossen
3D Kicad Symbolpfade angepasst
Anmerkungen in Schaltplan zu den Änderungen der 1.4 Platine entfernt
Schaltplan als PDF erstellt
Datei Leichen in Archiv verschoben
Unterordner für Datenblättererstellt
Unterordner für Produktionsdaten erstellt
Schaltplan und Platinen Layout Kicad Format geändert (von Kicad automatisch geändert)
+ Am Schaltplan und dem Platinen Layout wurden keine Änderungen vorgenommen+
Parts:
- Q36: Bestücken (Assemble) JA (YES) -> (none); JLCPCB LCSC Part C8545 -> (none); Reichelt-Bestellnummer R: BSS 138 SMD -> (none)
- R121: Funktion SMD-Widerstand, 0603, 10 kOhm, 100 mW, 1% -> (none); Hersteller Value -> (none); Hersteller Bestellnummer Value -> (none); Reichelt-Bestellnummer R: RND 0603 1 10K -> (none)
- R122: Bestücken (Assemble) JA (YES) -> (none); Reichelt-Bestellnummer R: RND 0603 1 10K -> (none)
Other:
- note removed: "Konntrolieren ob Footprint und Lib passt"
