File: pcb/Test_und_Entwicklung/megashield_svn_1.4_Prototyp_Intern_geschlossen/MähmotorSchutz.kicad_sch (KiCad schematic)
At the start: 6 parts

Commit message: megashield_svn_1.4_Prototyp_Intern_geschlossen
megashield_svn_1.4_Prototyp_Intern_geschlossen
3D Kicad Symbolpfade angepasst
Anmerkungen in Schaltplan zu den Änderungen der 1.4 Platine entfernt
Schaltplan als PDF erstellt
Datei Leichen in Archiv verschoben
Unterordner für Datenblättererstellt
Unterordner für Produktionsdaten erstellt
Schaltplan und Platinen Layout Kicad Format geändert (von Kicad automatisch geändert)
+ Am Schaltplan und dem Platinen Layout wurden keine Änderungen vorgenommen+
Parts:
- BY1, BY2, BY4: Bestücken (Assemble) JA (YES) -> (none); Funktion Gleichrichter 1000V 5A -> (none); Hersteller Nummer S5MC-13-F -> (none); Mouser Datenblatt https://www.mouser.de/datasheet/2/115/ds16007-37966.pdf -> (none); Mouser Nummer 621-S5MC-F -> (none)
- BY3: Bestücken (Assemble) JA (YES) -> (none); Hersteller Nummer S5MC-13-F -> (none); JLCPCB LCSC Part C123929 -> (none); Mouser Datenblatt https://www.mouser.de/datasheet/2/115/ds16007-37966.pdf -> (none); Mouser Nummer 621-S5MC-F -> (none)
- CC1: Bestellnummer Value -> (none); Bestücken (Assemble) JA (YES) -> (none); JLCPCB Basic / Extern 1 -> (none)
- RL1: Bestelllink https://www.tme.eu/en/details/wf25p-1r8-5%25/2512-smd-resis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 -> (none); Gehäuseart 2512 -> (none); JLCPCB Basic / Extern 1 -> (none)
Changed lines of the file:
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@@
-(kicad_sch (version 20201015) (generator eeschema)
+(kicad_sch (version 20210406) (generator eeschema)
   (paper "A4")
   (title_block
@@
     (property "Footprint" "" (id 2) (at 80.518 112.903 0))
     (property "Datasheet" "" (id 3) (at 80.518 112.903 0))
+    (pin "1")
   )
   (symbol (lib_id "ardumower-mega-shield-svn-rescue:GND-RESCUE-ardumower_mega_shield_svn") (at 124.333 112.903 0) (unit 1)
@@
     (property "Footprint" "" (id 2) (at 124.333 112.903 0))
     (property "Datasheet" "" (id 3) (at 124.333 112.903 0))
+    (pin "1")
   )
   (symbol (lib_id "ardumower-mega-shield-svn-rescue:R-RESCUE-ardumower_mega_shield_svn") (at 110.49 98.298 90) (unit 1)
@@
       (effects (font (size 1.27 1.27)) hide)
     )
-    (property "Bestelllink" "https://www.tme.eu/en/details/wf25p-1r8-5%25/2512-smd-resistors/walsin/wf25p1r8jtl/" (id 4) (at 110.49 98.298 0)
-      (effects (font (size 1.27 1.27)) hide)
-    )
-    (property "Gehäuseart" "2512" (id 5) (at 110.49 98.298 0)
-      (effects (font (size 1.27 1.27)) hide)
-    )
-    (property "JLCPCB Basic / Extern" "1" (id 6) (at 110.49 98.298 0)
-      (effects (font (size 1.27 1.27)) hide)
-    )
-    (property "JLCPCB LCSC Part" "C25473" (id 7) (at 110.49 98.298 0)
-      (effects (font (size 1.27 1.27)) hide)
-    )
+    (property "JLCPCB LCSC Part" "C25473" (id 8) (at 110.49 98.298 0)
+      (effects (font (size 1.27 1.27)) hide)
+    )
+    (pin "1")
+    (pin "2")
   )
   (symbol (lib_id "ardumower-mega-shield-svn-rescue:D-RESCUE-ardumower_mega_shield_svn") (at 80.518 90.551 90) (mirror x) (unit 1)
@@
       (effects (font (size 1.27 1.27)) hide)
     )
-    (property "Funktion" "Gleichrichter 1000V 5A" (id 4) (at 80.518 90.551 0)
-      (effects (font (size 1.27 1.27)) hide)
-    )
-    (property "Hersteller Nummer" "S5MC-13-F " (id 5) (at 80.518 90.551 0)
-      (effects (font (size 1.27 1.27)) hide)
-    )
-    (property "Mouser Datenblatt" "https://www.mouser.de/datasheet/2/115/ds16007-37966.pdf" (id 6) (at 80.518 90.551 0)
-      (effects (font (size 1.27 1.27)) hide)
-    )
-    (property "Mouser Nummer" "621-S5MC-F " (id 7) (at 80.518 90.551 0)
-      (effects (font (size 1.27 1.27)) hide)
-    )
-    (property "Bestücken (Assemble)" "JA (YES)" (id 8) (at 80.518 90.551 0)
-      (effects (font (size 1.27 1.27)) hide)
-    )
-    (property "JLCPCB Basic / Extern" "1" (id 9) (at 80.518 90.551 0)
-      (effects (font (size 1.27 1.27)) hide)
-    )
+    (property "JLCPCB Basic / Extern" "1" (id 10) (at 80.518 90.551 0)
+      (effects (font (size 1.27 1.27)) hide)
+    )
+    (pin "1")
+    (pin "2")
   )
   (symbol (lib_id "ardumower-mega-shield-svn-rescue:D-RESCUE-ardumower_mega_shield_svn") (at 80.518 104.902 270) (unit 1)
@@
       (effects (font (size 1.27 1.27)) hide)
     )
-    (property "Funktion" "Gleichrichter 1000V 5A" (id 4) (at 80.518 104.902 0)
-      (effects (font (size 1.27 1.27)) hide)
-    )
-    (property "Hersteller Nummer" "S5MC-13-F " (id 5) (at 80.518 104.902 0)
-      (effects (font (size 1.27 1.27)) hide)
-    )
-    (property "Mouser Datenblatt" "https://www.mouser.de/datasheet/2/115/ds16007-37966.pdf" (id 6) (at 80.518 104.902 0)
-      (effects (font (size 1.27 1.27)) hide)
-    )
-    (property "Mouser Nummer" "621-S5MC-F " (id 7) (at 80.518 104.902 0)
-      (effects (font (size 1.27 1.27)) hide)
-    )
-    (property "Bestücken (Assemble)" "JA (YES)" (id 8) (at 80.518 104.902 0)
-      (effects (font (size 1.27 1.27)) hide)
-    )
-    (property "JLCPCB Basic / Extern" "1" (id 9) (at 80.518 104.902 0)
-      (effects (font (size 1.27 1.27)) hide)
-    )
+    (property "JLCPCB Basic / Extern" "1" (id 10) (at 80.518 104.902 0)
+      (effects (font (size 1.27 1.27)) hide)
+    )
+    (pin "1")
+    (pin "2")
   )
   (symbol (lib_id "ardumower-mega-shield-svn-rescue:D-RESCUE-ardumower_mega_shield_svn") (at 124.333 91.059 270) (unit 1)
@@
       (effects (font (size 1.524 1.524)) hide)
     )
-    (property "Bestücken (Assemble)" "JA (YES)" (id 4) (at 124.333 91.059 0)
-      (effects (font (size 1.27 1.27)) hide)
-    )
-    (property "Hersteller Nummer" "S5MC-13-F " (id 5) (at 124.333 91.059 0)
-      (effects (font (size 1.27 1.27)) hide)
-    )
-    (property "Mouser Datenblatt" "https://www.mouser.de/datasheet/2/115/ds16007-37966.pdf" (id 6) (at 124.333 91.059 0)
-      (effects (font (size 1.27 1.27)) hide)
-    )
-    (property "Mouser Nummer" "621-S5MC-F " (id 7) (at 124.333 91.059 0)
-      (effects (font (size 1.27 1.27)) hide)
-    )
-    (property "JLCPCB LCSC Part" "C123929" (id 8) (at 124.333 91.059 0)
-      (effects (font (size 1.27 1.27)) hide)
-    )
-    (property "JLCPCB Basic / Extern" "1" (id 9) (at 124.333 91.059 0)
-      (effects (font (size 1.27 1.27)) hide)
-    )
+    (property "JLCPCB Basic / Extern" "1" (id 12) (at 124.333 91.059 0)
+      (effects (font (size 1.27 1.27)) hide)
+    )
+    (pin "1")
+    (pin "2")
   )
   (symbol (lib_id "ardumower-mega-shield-svn-rescue:D-RESCUE-ardumower_mega_shield_svn") (at 124.333 104.902 270) (unit 1)
@@
       (effects (font (size 1.27 1.27)) hide)
     )
-    (property "Funktion" "Gleichrichter 1000V 5A" (id 4) (at 124.333 104.902 0)
-      (effects (font (size 1.27 1.27)) hide)
-    )
-    (property "Hersteller Nummer" "S5MC-13-F " (id 5) (at 124.333 104.902 0)
-      (effects (font (size 1.27 1.27)) hide)
-    )
-    (property "Mouser Datenblatt" "https://www.mouser.de/datasheet/2/115/ds16007-37966.pdf" (id 6) (at 124.333 104.902 0)
-      (effects (font (size 1.27 1.27)) hide)
-    )
-    (property "Mouser Nummer" "621-S5MC-F " (id 7) (at 124.333 104.902 0)
-      (effects (font (size 1.27 1.27)) hide)
-    )
-    (property "Bestücken (Assemble)" "JA (YES)" (id 8) (at 124.333 104.902 0)
-      (effects (font (size 1.27 1.27)) hide)
-    )
-    (property "JLCPCB Basic / Extern" "1" (id 9) (at 124.333 104.902 0)
-      (effects (font (size 1.27 1.27)) hide)
-    )
+    (property "JLCPCB Basic / Extern" "1" (id 10) (at 124.333 104.902 0)
+      (effects (font (size 1.27 1.27)) hide)
+    )
+    (pin "1")
+    (pin "2")
   )
   (symbol (lib_id "ardumower-mega-shield-svn-rescue:C-RESCUE-ardumower_mega_shield_svn") (at 91.948 98.298 90) (unit 1)
@@
       (effects (font (size 1.27 1.27)) hide)
     )
-    (property "Bestücken (Assemble)" "JA (YES)" (id 4) (at 91.948 98.298 0)
-      (effects (font (size 1.27 1.27)) hide)
-    )
-    (property "Bestellnummer" "Value" (id 5) (at 91.948 98.298 0)
-      (effects (font (size 1.27 1.27)) hide)
-    )
-    (property "JLCPCB Basic / Extern" "1" (id 6) (at 91.948 98.298 0)
-      (effects (font (size 1.27 1.27)) hide)
-    )
-    (property "JLCPCB LCSC Part" "C1944" (id 7) (at 91.948 98.298 0)
-      (effects (font (size 1.27 1.27)) hide)
-    )
+    (property "JLCPCB LCSC Part" "C1944" (id 9) (at 91.948 98.298 0)
+      (effects (font (size 1.27 1.27)) hide)
+    )
+    (pin "1")
+    (pin "2")
   )
 )
