File: pcb/Test_und_Entwicklung/megashield_svn_1.4_Prototyp_Intern_geschlossen/Stromsensor_INA.kicad_sch (KiCad schematic)
At the start: 6 parts

Commit message: megashield_svn_1.4_Prototyp_Intern_geschlossen
megashield_svn_1.4_Prototyp_Intern_geschlossen
3D Kicad Symbolpfade angepasst
Anmerkungen in Schaltplan zu den Änderungen der 1.4 Platine entfernt
Schaltplan als PDF erstellt
Datei Leichen in Archiv verschoben
Unterordner für Datenblättererstellt
Unterordner für Produktionsdaten erstellt
Schaltplan und Platinen Layout Kicad Format geändert (von Kicad automatisch geändert)
+ Am Schaltplan und dem Platinen Layout wurden keine Änderungen vorgenommen+
Parts:
- C37: Bestücken (Assemble) JA (YES) -> (none)
- I1: JLCPCB Basic / Extern 1 -> (none)
- R138: Bestücken (Assemble) JA (YES) -> (none); Reichelt-Bestellnummer R: SPR-0603 6,80K -> (none)
- R139: Bestücken (Assemble) JA (YES) -> (none); Reichelt-Bestellnummer R: SPR-0603 3,30K -> (none)
- R140: Bestücken (Assemble) JA (YES) -> (none); Hersteller Nummer RCWE251250L0FKEA -> (none); JLCPCB Basic / Extern 1 -> (none); Mouser Datenblatt https://www.mouser.de/datasheet/2/427/rcwe-1761813.pdf -> (none); Mouser Nummer 71-RCWE251250L0FKEA -> (none)
